Commit message: imporve the scale of the model, add a laser, add a topic of the laser, can view it in gazebo in rviz, can mesure the object nearly

File: workspace/src/car_description/urdf/car.plugin.xacro (robot description, xacro)
@@ -2,34 +2,38 @@
 <robot>
 <!-- Laser sensor plugin -->
-  <gazebo reference="laser_1">
-    <sensor type="gpu_ray" name="head_hokuyo_sensor">
+  <gazebo reference="Laser_1">
+    <sensor type="gpu_ray" name="laser_sensor">
       <pose>0 0 0 0 0 0</pose>
       <visualize>true</visualize>
-      <update_rate>30</update_rate>
+      <update_rate>10.0</update_rate>
       <ray>
         <scan>
           <horizontal>
-            <samples>720</samples>
+            <samples>360</samples>
             <resolution>1</resolution>
-            <min_angle>-1.57</min_angle> <!-- -90 degrees -->
-            <max_angle>1.57</max_angle>  <!-- 90 degrees -->
+            <min_angle>-3.14</min_angle> <!-- -180 degrees -->
+            <max_angle>3.14</max_angle>  <!-- 180 degrees -->
           </horizontal>
+          <vertical>
+            <samples>30</samples> <!-- Número de "líneas" verticales que va a capturar -->
+            <min_angle>-0.3</min_angle> <!-- Ajusta el ángulo mínimo vertical -->
+            <max_angle>0.3</max_angle>  <!-- Ajusta el ángulo máximo vertical -->
+          </vertical>
         </scan>
         <range>
-          <min>0.1</min>  <!-- Minimum distance in meters -->
-          <max>10.0</max> <!-- Maximum distance in meters -->
+          <min>0.1</min>
+          <max>10.0</max>
           <resolution>0.01</resolution>
         </range>
         <noise>
-            <type>gaussian</type>
-            <mean>0.0</mean>
-            <stddev>0.01</stddev>
+          <type>gaussian</type>
+          <mean>0.0</mean>
+          <stddev>0.01</stddev>
         </noise>
       </ray>
-      <plugin name="gazebo_ros_head_hokuyo_controller"
-        filename="libgazebo_ros_ray_sensor.so">
-        <topicName>scan</topicName> <!-- Remap scan topic -->
-        <frameName>laser_1</frameName> <!-- Frame link for laser -->
-        <output_type>sensor_msgs/LaserScan</output_type>
+      <plugin name="gazebo_ros_laser" filename="libgazebo_ros_ray_sensor.so">
+        <topicName>/scan</topicName>
+        <frameName>Laser_1</frameName>
+        <output_type>sensor_msgs/PointCloud2</output_type>
       </plugin>
     </sensor>

File: workspace/src/car_description/urdf/car.xacro (robot description, xacro)
@@ -7,7 +7,7 @@
 <link name="base_link">
   <inertial>
-    <origin xyz="0.02503210561392206 -0.01250000000041644 0.0035096585129147538" rpy="0 0 0"/>
-    <mass value="0.06894028040642299"/>
-    <inertia ixx="4e-06" iyy="1.5e-05" izz="1.8e-05" ixy="0.0" iyz="0.0" ixz="-0.0"/>
+    <origin xyz="0.500073167158104 0.25000000000000006 0.25004231448306036" rpy="0 0 0"/>
+    <mass value="1963.3569872059904"/>
+    <inertia ixx="81.833055" iyy="204.557202" izz="204.546447" ixy="0.0" iyz="0.0" ixz="-0.036262"/>
   </inertial>
   <visual>
@@ -25,132 +25,132 @@
   </collision>
 </link>
-<link name="wheel_right_back_1">
+<link name="Wheel_front_right_1">
   <inertial>
-    <origin xyz="1.1920929174347172e-10 -0.0035000000000000066 5.9604635463395e-11" rpy="0 0 0"/>
-    <mass value="0.00621469877254378"/>
-    <inertia ixx="0.0" iyy="0.0" izz="0.0" ixy="0.0" iyz="0.0" ixz="-0.0"/>
+    <origin xyz="0.0 -0.05000000000000001 0.0" rpy="0 0 0"/>
+    <mass value="98.6460093227195"/>
+    <inertia ixx="1.068665" iyy="1.97292" izz="1.068665" ixy="-0.0" iyz="-0.0" ixz="0.0"/>
   </inertial>
   <visual>
-    <origin xyz="-0.008 0.026 -0.004" rpy="0 0 0"/>
+    <origin xyz="-0.875 0.01 -0.15" rpy="0 0 0"/>
     <geometry>
-      <mesh filename="file://$(find car_description)/meshes/wheel_right_back_1.stl" scale="0.001 0.001 0.001"/>
+      <mesh filename="file://$(find car_description)/meshes/Wheel_front_right_1.stl" scale="0.001 0.001 0.001"/>
     </geometry>
     <material name="silver"/>
   </visual>
   <collision>
-    <origin xyz="-0.008 0.026 -0.004" rpy="0 0 0"/>
+    <origin xyz="-0.875 0.01 -0.15" rpy="0 0 0"/>
     <geometry>
-      <mesh filename="file://$(find car_description)/meshes/wheel_right_back_1.stl" scale="0.001 0.001 0.001"/>
+      <mesh filename="file://$(find car_description)/meshes/Wheel_front_right_1.stl" scale="0.001 0.001 0.001"/>
     </geometry>
   </collision>
 </link>
-<link name="wheel_right_front_1">
+<link name="Wheel_front_left_1">
   <inertial>
-    <origin xyz="5.960464413701239e-10 -0.0035000000000000135 5.960463719811848e-11" rpy="0 0 0"/>
-    <mass value="0.006214698772543783"/>
-    <inertia ixx="0.0" iyy="0.0" izz="0.0" ixy="-0.0" iyz="0.0" ixz="0.0"/>
+    <origin xyz="0.0 0.050000000000000044 0.0" rpy="0 0 0"/>
+    <mass value="98.6460093227195"/>
+    <inertia ixx="1.068665" iyy="1.97292" izz="1.068665" ixy="0.0" iyz="0.0" ixz="0.0"/>
   </inertial>
   <visual>
-    <origin xyz="-0.04 0.026 -0.004" rpy="0 0 0"/>
+    <origin xyz="-0.875 -0.51 -0.15" rpy="0 0 0"/>
     <geometry>
-      <mesh filename="file://$(find car_description)/meshes/wheel_right_front_1.stl" scale="0.001 0.001 0.001"/>
+      <mesh filename="file://$(find car_description)/meshes/Wheel_front_left_1.stl" scale="0.001 0.001 0.001"/>
     </geometry>
     <material name="silver"/>
   </visual>
   <collision>
-    <origin xyz="-0.04 0.026 -0.004" rpy="0 0 0"/>
+    <origin xyz="-0.875 -0.51 -0.15" rpy="0 0 0"/>
     <geometry>
-      <mesh filename="file://$(find car_description)/meshes/wheel_right_front_1.stl" scale="0.001 0.001 0.001"/>
+      <mesh filename="file://$(find car_description)/meshes/Wheel_front_left_1.stl" scale="0.001 0.001 0.001"/>
     </geometry>
   </collision>
 </link>
-<link name="wheel_left_front_1">
+<link name="Wheel_back_left_1">
   <inertial>
-    <origin xyz="5.960464483090178e-10 0.0034999999999999988 5.96046467390976e-11" rpy="0 0 0"/>
-    <mass value="0.006214698772543782"/>
-    <inertia ixx="0.0" iyy="0.0" izz="0.0" ixy="0.0" iyz="-0.0" ixz="-0.0"/>
+    <origin xyz="-2.7755575615628914e-17 0.050000000000000155 0.0" rpy="0 0 0"/>
+    <mass value="98.6460093227195"/>
+    <inertia ixx="1.068665" iyy="1.97292" izz="1.068665" ixy="0.0" iyz="0.0" ixz="0.0"/>
   </inertial>
   <visual>
-    <origin xyz="-0.04 -0.001 -0.004" rpy="0 0 0"/>
+    <origin xyz="-0.15 -0.51 -0.15" rpy="0 0 0"/>
     <geometry>
-      <mesh filename="file://$(find car_description)/meshes/wheel_left_front_1.stl" scale="0.001 0.001 0.001"/>
+      <mesh filename="file://$(find car_description)/meshes/Wheel_back_left_1.stl" scale="0.001 0.001 0.001"/>
     </geometry>
     <material name="silver"/>
   </visual>
   <collision>
-    <origin xyz="-0.04 -0.001 -0.004" rpy="0 0 0"/>
+    <origin xyz="-0.15 -0.51 -0.15" rpy="0 0 0"/>
     <geometry>
-      <mesh filename="file://$(find car_description)/meshes/wheel_left_front_1.stl" scale="0.001 0.001 0.001"/>
+      <mesh filename="file://$(find car_description)/meshes/Wheel_back_left_1.stl" scale="0.001 0.001 0.001"/>
     </geometry>
   </collision>
 </link>
-<link name="wheel_left_back_1">
+<link name="Wheel_back_right_1">
   <inertial>
-    <origin xyz="1.1920929000874825e-10 0.0034999999999999996 5.960464500437412e-11" rpy="0 0 0"/>
-    <mass value="0.006214698772543781"/>
-    <inertia ixx="0.0" iyy="0.0" izz="0.0" ixy="-0.0" iyz="0.0" ixz="-0.0"/>
+    <origin xyz="-2.7755575615628914e-17 -0.05000000000000001 0.0" rpy="0 0 0"/>
+    <mass value="98.6460093227195"/>
+    <inertia ixx="1.068665" iyy="1.97292" izz="1.068665" ixy="0.0" iyz="-0.0" ixz="0.0"/>
   </inertial>
   <visual>
-    <origin xyz="-0.008 -0.001 -0.004" rpy="0 0 0"/>
+    <origin xyz="-0.15 0.01 -0.15" rpy="0 0 0"/>
     <geometry>
-      <mesh filename="file://$(find car_description)/meshes/wheel_left_back_1.stl" scale="0.001 0.001 0.001"/>
+      <mesh filename="file://$(find car_description)/meshes/Wheel_back_right_1.stl" scale="0.001 0.001 0.001"/>
     </geometry>
     <material name="silver"/>
   </visual>
   <collision>
-    <origin xyz="-0.008 -0.001 -0.004" rpy="0 0 0"/>
+    <origin xyz="-0.15 0.01 -0.15" rpy="0 0 0"/>
     <geometry>
-      <mesh filename="file://$(find car_description)/meshes/wheel_left_back_1.stl" scale="0.001 0.001 0.001"/>
+      <mesh filename="file://$(find car_description)/meshes/Wheel_back_right_1.stl" scale="0.001 0.001 0.001"/>
     </geometry>
   </collision>
 </link>
-<link name="laser_1">
+<link name="Laser_1">
   <inertial>
-    <origin xyz="5.960464552479117e-10 -1.862645159639298e-10 0.0024999999999999953" rpy="0 0 0"/>
-    <mass value="0.004439070551816985"/>
-    <inertia ixx="0.0" iyy="0.0" izz="0.0" ixy="0.0" iyz="0.0" ixz="-0.0"/>
+    <origin xyz="-2.220446049250313e-16 5.551115123125783e-17 0.03499999999999992" rpy="0 0 0"/>
+    <mass value="52.86809562139498"/>
+    <inertia ixx="0.426359" iyy="0.426359" izz="0.809543" ixy="0.0" iyz="-0.0" ixz="0.0"/>
   </inertial>
   <visual>
-    <origin xyz="-0.04 0.0125 -0.008" rpy="0 0 0"/>
+    <origin xyz="-0.8 -0.25 -0.53" rpy="0 0 0"/>
     <geometry>
-      <mesh filename="file://$(find car_description)/meshes/laser_1.stl" scale="0.001 0.001 0.001"/>
+      <mesh filename="file://$(find car_description)/meshes/Laser_1.stl" scale="0.001 0.001 0.001"/>
     </geometry>
     <material name="silver"/>
   </visual>
   <collision>
-    <origin xyz="-0.04 0.0125 -0.008" rpy="0 0 0"/>
+    <origin xyz="-0.8 -0.25 -0.53" rpy="0 0 0"/>
     <geometry>
-      <mesh filename="file://$(find car_description)/meshes/laser_1.stl" scale="0.001 0.001 0.001"/>
+      <mesh filename="file://$(find car_description)/meshes/Laser_1.stl" scale="0.001 0.001 0.001"/>
     </geometry>
   </collision>
 </link>
-<joint name="Revolute 9" type="continuous">
-  <origin xyz="0.008 -0.026 0.004" rpy="0 0 0"/>
+<joint name="revolute_right_wheel" type="continuous">
+  <origin xyz="0.875 -0.01 0.15" rpy="0 0 0"/>
   <parent link="base_link"/>
-  <child link="wheel_right_back_1"/>
+  <child link="Wheel_front_right_1"/>
   <axis xyz="0.0 -1.0 0.0"/>
 </joint>
-<joint name="Revolute 10" type="continuous">
-  <origin xyz="0.04 -0.026 0.004" rpy="0 0 0"/>
+<joint name="revolute_left_wheel" type="continuous">
+  <origin xyz="0.875 0.51 0.15" rpy="0 0 0"/>
   <parent link="base_link"/>
-  <child link="wheel_right_front_1"/>
+  <child link="Wheel_front_left_1"/>
+  <axis xyz="0.0 1.0 0.0"/>
+</joint>
+<joint name="revolute_back_left_wheel" type="continuous">
+  <origin xyz="0.15 0.51 0.15" rpy="0 0 0"/>
+  <parent link="base_link"/>
+  <child link="Wheel_back_left_1"/>
+  <axis xyz="0.0 1.0 0.0"/>
+</joint>
+<joint name="revolute_back_right_wheel" type="continuous">
+  <origin xyz="0.15 -0.01 0.15" rpy="0 0 0"/>
+  <parent link="base_link"/>
+  <child link="Wheel_back_right_1"/>
   <axis xyz="0.0 -1.0 0.0"/>
 </joint>
-<joint name="Revolute 11" type="continuous">
-  <origin xyz="0.04 0.001 0.004" rpy="0 0 0"/>
+<joint name="revolute_laser" type="continuous">
+  <origin xyz="0.8 0.25 0.53" rpy="0 0 0"/>
   <parent link="base_link"/>
-  <child link="wheel_left_front_1"/>
-  <axis xyz="0.0 1.0 0.0"/>
-</joint>
-<joint name="Revolute 12" type="continuous">
-  <origin xyz="0.008 0.001 0.004" rpy="0 0 0"/>
-  <parent link="base_link"/>
-  <child link="wheel_left_back_1"/>
-  <axis xyz="0.0 1.0 0.0"/>
-</joint>
-<joint name="Revolute 13" type="continuous">
-  <origin xyz="0.04 -0.0125 0.008" rpy="0 0 0"/>
-  <parent link="base_link"/>
-  <child link="laser_1"/>
+  <child link="Laser_1"/>
   <axis xyz="0.0 0.0 1.0"/>
 </joint>
