Commit message: new model of the robot,new world and launch for each worl even the empty world, add a depth camera and his frame for rviz

File: workspace/src/car/urdf/car.plugin.xacro (robot description, xacro)
@@ -5,5 +5,5 @@
     <sensor type="gpu_ray" name="laser_sensor">
       <pose>0 0 0 0 0 0</pose>
-      <visualize>true</visualize>
+      <visualize>false</visualize>
       <update_rate>30.0</update_rate>
       <ray>
@@ -33,6 +33,5 @@
       </ray>
       <plugin name="gazebo_ros_laser" filename="libgazebo_ros_ray_sensor.so">
-        <topicName>/scan</topicName>
-        <frameName>Laser_1</frameName>
+        <frame_name>base_link</frame_name>
         <!-- <output_type>sensor_msgs/PointCloud2</output_type> -->
       </plugin>

File: workspace/src/car/urdf/car.xacro (robot description, xacro)
@@ -5,9 +5,10 @@
 <xacro:include filename="$(find car)/urdf/car.gazebo" />
 <xacro:include filename="$(find car)/urdf/car.plugin.xacro" />
+<xacro:include filename="$(find car)/urdf/depth.plugin.xacro" />
 <link name="base_link">
   <inertial>
-    <origin xyz="0.500073167158104 0.25000000000000006 0.25004231448306036" rpy="0 0 0"/>
-    <mass value="1963.3569872059904"/>
-    <inertia ixx="81.833055" iyy="204.557202" izz="204.546447" ixy="0.0" iyz="0.0" ixz="-0.036262"/>
+    <origin xyz="0.5000181378162949 0.25000000000000006 0.2517249688727959" rpy="0 0 0"/>
+    <mass value="1971.5261098530282"/>
+    <inertia ixx="83.35609" iyy="206.212802" izz="204.780211" ixy="0.0" iyz="0.0" ixz="-0.007768"/>
   </inertial>
   <visual>
@@ -107,10 +108,10 @@
 <link name="Laser_1">
   <inertial>
-    <origin xyz="-2.220446049250313e-16 5.551115123125783e-17 0.03499999999999992" rpy="0 0 0"/>
-    <mass value="52.86809562139498"/>
-    <inertia ixx="0.426359" iyy="0.426359" izz="0.809543" ixy="0.0" iyz="-0.0" ixz="0.0"/>
-  </inertial>
-  <visual>
-    <origin xyz="-0.8 -0.25 -0.53" rpy="0 0 0"/>
+    <origin xyz="1.1102230246251565e-16 -2.7755575615628914e-17 0.015000000000000013" rpy="0 0 0"/>
+    <mass value="7.398450699203962"/>
+    <inertia ixx="0.019051" iyy="0.019051" izz="0.036992" ixy="0.0" iyz="0.0" ixz="0.0"/>
+  </inertial>
+  <visual>
+    <origin xyz="-0.5 -0.25 -0.9" rpy="0 0 0"/>
     <geometry>
       <mesh filename="file://$(find car)/meshes/Laser_1.stl" scale="0.001 0.001 0.001"/>
@@ -119,7 +120,87 @@
   </visual>
   <collision>
-    <origin xyz="-0.8 -0.25 -0.53" rpy="0 0 0"/>
+    <origin xyz="-0.5 -0.25 -0.9" rpy="0 0 0"/>
     <geometry>
       <mesh filename="file://$(find car)/meshes/Laser_1.stl" scale="0.001 0.001 0.001"/>
+    </geometry>
+  </collision>
+</link>
+<link name="Camara_back_1">
+  <inertial>
+    <origin xyz="6.938893903907228e-17 -2.7755575615628914e-17 0.015000000000000013" rpy="0 0 0"/>
+    <mass value="7.398450699203962"/>
+    <inertia ixx="0.019051" iyy="0.019051" izz="0.036992" ixy="-0.0" iyz="0.0" ixz="-0.0"/>
+  </inertial>
+  <visual>
+    <origin xyz="-0.1 -0.25 -0.54" rpy="0 0 0"/>
+    <geometry>
+      <mesh filename="file://$(find car)/meshes/Camara_back_1.stl" scale="0.001 0.001 0.001"/>
+    </geometry>
+    <material name="silver"/>
+  </visual>
+  <collision>
+    <origin xyz="-0.1 -0.25 -0.54" rpy="0 0 0"/>
+    <geometry>
+      <mesh filename="file://$(find car)/meshes/Camara_back_1.stl" scale="0.001 0.001 0.001"/>
+    </geometry>
+  </collision>
+</link>
+<link name="Camara_left_1">
+  <inertial>
+    <origin xyz="-5.551115123125783e-17 0.0 0.015000000000000013" rpy="0 0 0"/>
+    <mass value="7.398450699203962"/>
+    <inertia ixx="0.019051" iyy="0.019051" izz="0.036992" ixy="0.0" iyz="0.0" ixz="0.0"/>
+  </inertial>
+  <visual>
+    <origin xyz="-0.5 -0.45 -0.54" rpy="0 0 0"/>
+    <geometry>
+      <mesh filename="file://$(find car)/meshes/Camara_left_1.stl" scale="0.001 0.001 0.001"/>
+    </geometry>
+    <material name="silver"/>
+  </visual>
+  <collision>
+    <origin xyz="-0.5 -0.45 -0.54" rpy="0 0 0"/>
+    <geometry>
+      <mesh filename="file://$(find car)/meshes/Camara_left_1.stl" scale="0.001 0.001 0.001"/>
+    </geometry>
+  </collision>
+</link>
+<link name="Camara_front_1">
+  <inertial>
+    <origin xyz="0.0 -2.7755575615628914e-17 0.015000000000000013" rpy="0 0 0"/>
+    <mass value="7.398450699203962"/>
+    <inertia ixx="0.019051" iyy="0.019051" izz="0.036992" ixy="0.0" iyz="0.0" ixz="0.0"/>
+  </inertial>
+  <visual>
+    <origin xyz="-0.95 -0.25 -0.54" rpy="0 0 0"/>
+    <geometry>
+      <mesh filename="file://$(find car)/meshes/Camara_front_1.stl" scale="0.001 0.001 0.001"/>
+    </geometry>
+    <material name="silver"/>
+  </visual>
+  <collision>
+    <origin xyz="-0.95 -0.25 -0.54" rpy="0 0 0"/>
+    <geometry>
+      <mesh filename="file://$(find car)/meshes/Camara_front_1.stl" scale="0.001 0.001 0.001"/>
+    </geometry>
+  </collision>
+</link>
+<link name="Camara_right_1">
+  <inertial>
+    <origin xyz="1.1102230246251565e-16 -1.3877787807814457e-17 0.015000000000000013" rpy="0 0 0"/>
+    <mass value="7.398450699203962"/>
+    <inertia ixx="0.019051" iyy="0.019051" izz="0.036992" ixy="0.0" iyz="0.0" ixz="0.0"/>
+  </inertial>
+  <visual>
+    <origin xyz="-0.5 -0.05 -0.54" rpy="0 0 0"/>
+    <geometry>
+      <mesh filename="file://$(find car)/meshes/Camara_right_1.stl" scale="0.001 0.001 0.001"/>
+    </geometry>
+    <material name="silver"/>
+  </visual>
+  <collision>
+    <origin xyz="-0.5 -0.05 -0.54" rpy="0 0 0"/>
+    <geometry>
+      <mesh filename="file://$(find car)/meshes/Camara_right_1.stl" scale="0.001 0.001 0.001"/>
     </geometry>
   </collision>
@@ -150,8 +231,40 @@
 </joint>
 <joint name="revolute_laser" type="continuous">
-  <origin xyz="0.8 0.25 0.53" rpy="0 0 0"/>
+  <origin xyz="0.5 0.25 0.9" rpy="0 0 0"/>
   <parent link="base_link"/>
   <child link="Laser_1"/>
   <axis xyz="0.0 0.0 1.0"/>
 </joint>
+<joint name="revolute_camara_back" type="continuous">
+  <origin xyz="0.1 0.25 0.54" rpy="0 0 0"/>
+  <parent link="base_link"/>
+  <child link="Camara_back_1"/>
+  <axis xyz="0.0 0.0 1.0"/>
+</joint>
+<joint name="revoute_camara_left" type="continuous">
+  <origin xyz="0.5 0.45 0.54" rpy="0 0 0"/>
+  <parent link="base_link"/>
+  <child link="Camara_left_1"/>
+  <axis xyz="0.0 0.0 1.0"/>
+</joint>
+<joint name="revolute_camara_front" type="continuous">
+  <origin xyz="0.95 0.25 0.54" rpy="0 0 0"/>
+  <parent link="base_link"/>
+  <child link="Camara_front_1"/>
+  <axis xyz="0.0 0.0 1.0"/>
+</joint>
+<link name="camera_optical_frame">
+</link>
+<joint name="camera_optical_joint" type="fixed">
+  <parent link="Camara_front_1"/>
+  <child link="camera_optical_frame"/>
+  <!-- Ajusta rpy para alinear el frame óptico -->
+  <origin xyz="0 0 0" rpy="-1.5708 0 -1.5708"/>
+</joint>
+<joint name="revolute_camara_right" type="continuous">
+  <origin xyz="0.5 0.05 0.54" rpy="0 0 0"/>
+  <parent link="base_link"/>
+  <child link="Camara_right_1"/>
+  <axis xyz="0.0 0.0 1.0"/>
+</joint>
 </robot>
