Commit message: fixed the model?

File: workspace/src/car_python/urdf/car.xacro (robot description, xacro)
@@ -264,4 +264,124 @@
   </collision>
 </link>
+<link name="direction_front_right_1">
+  <inertial>
+    <origin xyz="0.00201472265142022 0.07474229529205378 5.551115123125783e-17" rpy="0 0 0"/>
+    <mass value="11.386858894419678"/>
+    <inertia ixx="0.054235" iyy="0.024154" izz="0.06804" ixy="-0.00144" iyz="0.0" ixz="0.0"/>
+  </inertial>
+  <visual>
+    <origin xyz="-0.575 -1.5875 0.45" rpy="0 0 0"/>
+    <geometry>
+      <mesh filename="file://$(find car_description)/meshes/direction_front_right_1.stl" scale="0.001 0.001 0.001"/>
+    </geometry>
+    <material name="silver"/>
+  </visual>
+  <collision>
+    <origin xyz="-0.575 -1.5875 0.45" rpy="0 0 0"/>
+    <geometry>
+      <mesh filename="file://$(find car_description)/meshes/direction_front_right_1.stl" scale="0.001 0.001 0.001"/>
+    </geometry>
+  </collision>
+</link>
+<link name="direction_front_left_1">
+  <inertial>
+    <origin xyz="0.002014722651420442 -0.07474229529205342 0.0" rpy="0 0 0"/>
+    <mass value="11.386858894419664"/>
+    <inertia ixx="0.054235" iyy="0.024154" izz="0.06804" ixy="0.00144" iyz="0.0" ixz="-0.0"/>
+  </inertial>
+  <visual>
+    <origin xyz="-0.575 0.0875 0.45" rpy="0 0 0"/>
+    <geometry>
+      <mesh filename="file://$(find car_description)/meshes/direction_front_left_1.stl" scale="0.001 0.001 0.001"/>
+    </geometry>
+    <material name="silver"/>
+  </visual>
+  <collision>
+    <origin xyz="-0.575 0.0875 0.45" rpy="0 0 0"/>
+    <geometry>
+      <mesh filename="file://$(find car_description)/meshes/direction_front_left_1.stl" scale="0.001 0.001 0.001"/>
+    </geometry>
+  </collision>
+</link>
+<link name="direction_back_left_1">
+  <inertial>
+    <origin xyz="-2.220446049250313e-16 -0.07474229529205345 0.0" rpy="0 0 0"/>
+    <mass value="11.386858894419674"/>
+    <inertia ixx="0.054235" iyy="0.024086" izz="0.067971" ixy="0.0" iyz="0.0" ixz="0.0"/>
+  </inertial>
+  <visual>
+    <origin xyz="-1.925 0.0875 0.45" rpy="0 0 0"/>
+    <geometry>
+      <mesh filename="file://$(find car_description)/meshes/direction_back_left_1.stl" scale="0.001 0.001 0.001"/>
+    </geometry>
+    <material name="silver"/>
+  </visual>
+  <collision>
+    <origin xyz="-1.925 0.0875 0.45" rpy="0 0 0"/>
+    <geometry>
+      <mesh filename="file://$(find car_description)/meshes/direction_back_left_1.stl" scale="0.001 0.001 0.001"/>
+    </geometry>
+  </collision>
+</link>
+<link name="direction_back_right_1">
+  <inertial>
+    <origin xyz="2.220446049250313e-16 0.07474229529205334 5.551115123125783e-17" rpy="0 0 0"/>
+    <mass value="11.386858894419714"/>
+    <inertia ixx="0.054235" iyy="0.024086" izz="0.067971" ixy="-0.0" iyz="0.0" ixz="-0.0"/>
+  </inertial>
+  <visual>
+    <origin xyz="-1.925 -1.5875 0.45" rpy="0 0 0"/>
+    <geometry>
+      <mesh filename="file://$(find car_description)/meshes/direction_back_right_1.stl" scale="0.001 0.001 0.001"/>
+    </geometry>
+    <material name="silver"/>
+  </visual>
+  <collision>
+    <origin xyz="-1.925 -1.5875 0.45" rpy="0 0 0"/>
+    <geometry>
+      <mesh filename="file://$(find car_description)/meshes/direction_back_right_1.stl" scale="0.001 0.001 0.001"/>
+    </geometry>
+  </collision>
+</link>
+<link name="Lidar_1">
+  <inertial>
+    <origin xyz="-6.661338147750939e-16 -1.1102230246251565e-16 0.04999999999999993" rpy="0 0 0"/>
+    <mass value="24.661502330679863"/>
+    <inertia ixx="0.082205" iyy="0.082205" izz="0.123308" ixy="-0.0" iyz="0.0" ixz="-0.0"/>
+  </inertial>
+  <visual>
+    <origin xyz="-1.85 -0.75 -0.7" rpy="0 0 0"/>
+    <geometry>
+      <mesh filename="file://$(find car_description)/meshes/Lidar_1.stl" scale="0.001 0.001 0.001"/>
+    </geometry>
+    <material name="silver"/>
+  </visual>
+  <collision>
+    <origin xyz="-1.85 -0.75 -0.7" rpy="0 0 0"/>
+    <geometry>
+      <mesh filename="file://$(find car_description)/meshes/Lidar_1.stl" scale="0.001 0.001 0.001"/>
+    </geometry>
+  </collision>
+</link>
+<link name="Camara_1">
+  <inertial>
+    <origin xyz="-0.004642640365980721 0.0 -0.0018567286993164678" rpy="0 0 0"/>
+    <mass value="3.1890625000000425"/>
+    <inertia ixx="0.031654" iyy="0.004179" izz="0.028666" ixy="0.0" iyz="0.0" ixz="0.001423"/>
+  </inertial>
+  <visual>
+    <origin xyz="-2.162084 -0.7625 -0.447483" rpy="0 0 0"/>
+    <geometry>
+      <mesh filename="file://$(find car_description)/meshes/Camara_1.stl" scale="0.001 0.001 0.001"/>
+    </geometry>
+    <material name="silver"/>
+  </visual>
+  <collision>
+    <origin xyz="-2.162084 -0.7625 -0.447483" rpy="0 0 0"/>
+    <geometry>
+      <mesh filename="file://$(find car_description)/meshes/Camara_1.stl" scale="0.001 0.001 0.001"/>
+    </geometry>
+  </collision>
+</link>
 <link name="chasis_1">
   <inertial>
@@ -281,124 +401,4 @@
     <geometry>
       <mesh filename="file://$(find car_description)/meshes/chasis_1.stl" scale="0.001 0.001 0.001"/>
-    </geometry>
-  </collision>
-</link>
-<link name="direction_front_right_1">
-  <inertial>
-    <origin xyz="0.00201472265142022 0.07474229529205378 5.551115123125783e-17" rpy="0 0 0"/>
-    <mass value="11.386858894419678"/>
-    <inertia ixx="0.054235" iyy="0.024154" izz="0.06804" ixy="-0.00144" iyz="0.0" ixz="0.0"/>
-  </inertial>
-  <visual>
-    <origin xyz="-0.575 -1.5875 0.45" rpy="0 0 0"/>
-    <geometry>
-      <mesh filename="file://$(find car_description)/meshes/direction_front_right_1.stl" scale="0.001 0.001 0.001"/>
-    </geometry>
-    <material name="silver"/>
-  </visual>
-  <collision>
-    <origin xyz="-0.575 -1.5875 0.45" rpy="0 0 0"/>
-    <geometry>
-      <mesh filename="file://$(find car_description)/meshes/direction_front_right_1.stl" scale="0.001 0.001 0.001"/>
-    </geometry>
-  </collision>
-</link>
-<link name="direction_front_left_1">
-  <inertial>
-    <origin xyz="0.002014722651420442 -0.07474229529205342 0.0" rpy="0 0 0"/>
-    <mass value="11.386858894419664"/>
-    <inertia ixx="0.054235" iyy="0.024154" izz="0.06804" ixy="0.00144" iyz="0.0" ixz="-0.0"/>
-  </inertial>
-  <visual>
-    <origin xyz="-0.575 0.0875 0.45" rpy="0 0 0"/>
-    <geometry>
-      <mesh filename="file://$(find car_description)/meshes/direction_front_left_1.stl" scale="0.001 0.001 0.001"/>
-    </geometry>
-    <material name="silver"/>
-  </visual>
-  <collision>
-    <origin xyz="-0.575 0.0875 0.45" rpy="0 0 0"/>
-    <geometry>
-      <mesh filename="file://$(find car_description)/meshes/direction_front_left_1.stl" scale="0.001 0.001 0.001"/>
-    </geometry>
-  </collision>
-</link>
-<link name="direction_back_left_1">
-  <inertial>
-    <origin xyz="-2.220446049250313e-16 -0.07474229529205345 0.0" rpy="0 0 0"/>
-    <mass value="11.386858894419674"/>
-    <inertia ixx="0.054235" iyy="0.024086" izz="0.067971" ixy="0.0" iyz="0.0" ixz="0.0"/>
-  </inertial>
-  <visual>
-    <origin xyz="-1.925 0.0875 0.45" rpy="0 0 0"/>
-    <geometry>
-      <mesh filename="file://$(find car_description)/meshes/direction_back_left_1.stl" scale="0.001 0.001 0.001"/>
-    </geometry>
-    <material name="silver"/>
-  </visual>
-  <collision>
-    <origin xyz="-1.925 0.0875 0.45" rpy="0 0 0"/>
-    <geometry>
-      <mesh filename="file://$(find car_description)/meshes/direction_back_left_1.stl" scale="0.001 0.001 0.001"/>
-    </geometry>
-  </collision>
-</link>
-<link name="direction_back_right_1">
-  <inertial>
-    <origin xyz="2.220446049250313e-16 0.07474229529205334 5.551115123125783e-17" rpy="0 0 0"/>
-    <mass value="11.386858894419714"/>
-    <inertia ixx="0.054235" iyy="0.024086" izz="0.067971" ixy="-0.0" iyz="0.0" ixz="-0.0"/>
-  </inertial>
-  <visual>
-    <origin xyz="-1.925 -1.5875 0.45" rpy="0 0 0"/>
-    <geometry>
-      <mesh filename="file://$(find car_description)/meshes/direction_back_right_1.stl" scale="0.001 0.001 0.001"/>
-    </geometry>
-    <material name="silver"/>
-  </visual>
-  <collision>
-    <origin xyz="-1.925 -1.5875 0.45" rpy="0 0 0"/>
-    <geometry>
-      <mesh filename="file://$(find car_description)/meshes/direction_back_right_1.stl" scale="0.001 0.001 0.001"/>
-    </geometry>
-  </collision>
-</link>
-<link name="Lidar_1">
-  <inertial>
-    <origin xyz="-6.661338147750939e-16 -1.1102230246251565e-16 0.04999999999999993" rpy="0 0 0"/>
-    <mass value="24.661502330679863"/>
-    <inertia ixx="0.082205" iyy="0.082205" izz="0.123308" ixy="-0.0" iyz="0.0" ixz="-0.0"/>
-  </inertial>
-  <visual>
-    <origin xyz="-1.85 -0.75 -0.7" rpy="0 0 0"/>
-    <geometry>
-      <mesh filename="file://$(find car_description)/meshes/Lidar_1.stl" scale="0.001 0.001 0.001"/>
-    </geometry>
-    <material name="silver"/>
-  </visual>
-  <collision>
-    <origin xyz="-1.85 -0.75 -0.7" rpy="0 0 0"/>
-    <geometry>
-      <mesh filename="file://$(find car_description)/meshes/Lidar_1.stl" scale="0.001 0.001 0.001"/>
-    </geometry>
-  </collision>
-</link>
-<link name="Camara_1">
-  <inertial>
-    <origin xyz="-0.004642640365980721 0.0 -0.0018567286993164678" rpy="0 0 0"/>
-    <mass value="3.1890625000000425"/>
-    <inertia ixx="0.031654" iyy="0.004179" izz="0.028666" ixy="0.0" iyz="0.0" ixz="0.001423"/>
-  </inertial>
-  <visual>
-    <origin xyz="-2.162084 -0.7625 -0.447483" rpy="0 0 0"/>
-    <geometry>
-      <mesh filename="file://$(find car_description)/meshes/Camara_1.stl" scale="0.001 0.001 0.001"/>
-    </geometry>
-    <material name="silver"/>
-  </visual>
-  <collision>
-    <origin xyz="-2.162084 -0.7625 -0.447483" rpy="0 0 0"/>
-    <geometry>
-      <mesh filename="file://$(find car_description)/meshes/Camara_1.stl" scale="0.001 0.001 0.001"/>
     </geometry>
   </collision>
@@ -476,9 +476,4 @@
   <child link="tire_front_left_1"/>
 </joint>
-<joint name="Rigid 13" type="fixed">
-  <origin xyz="1.25 0.75 -0.4" rpy="0 0 0"/>
-  <parent link="base_link"/>
-  <child link="chasis_1"/>
-</joint>
 <joint name="Revolute 14" type="revolute">
   <origin xyz="0.0 0.7125 0.0" rpy="0 0 0"/>
@@ -519,3 +514,8 @@
   <child link="Camara_1"/>
 </joint>
+<joint name="Rigid 20" type="fixed">
+  <origin xyz="1.25 0.75 -0.4" rpy="0 0 0"/>
+  <parent link="base_link"/>
+  <child link="chasis_1"/>
+</joint>
 </robot>
