Commit message: fixed the model finally

File: workspace/src/car_python/urdf/car.xacro (robot description, xacro)
@@ -1,7 +1,7 @@
 <?xml version="1.0" ?>
 <robot name="car" xmlns:xacro="http://www.ros.org/wiki/xacro">
-<xacro:include filename="$(find car_description)/urdf/materials.xacro" />
-<xacro:include filename="$(find car_description)/urdf/car.trans" />
-<xacro:include filename="$(find car_description)/urdf/car.gazebo" />
+<xacro:include filename="$(find car)/urdf/materials.xacro" />
+<xacro:include filename="$(find car)/urdf/car.trans" />
+<xacro:include filename="$(find car)/urdf/car.gazebo" />
 <link name="base_link">
   <inertial>
@@ -13,5 +13,5 @@
     <origin xyz="0 0 0" rpy="0 0 0"/>
     <geometry>
-      <mesh filename="file://$(find car_description)/meshes/base_link.stl" scale="0.001 0.001 0.001"/>
+      <mesh filename="file://$(find car)/meshes/base_link.stl" scale="0.001 0.001 0.001"/>
     </geometry>
     <material name="silver"/>
@@ -20,9 +20,9 @@
     <origin xyz="0 0 0" rpy="0 0 0"/>
     <geometry>
-      <mesh filename="file://$(find car_description)/meshes/base_link.stl" scale="0.001 0.001 0.001"/>
-    </geometry>
-  </collision>
-</link>
-<link name="suspension_back_left_1">
+      <mesh filename="file://$(find car)/meshes/base_link.stl" scale="0.001 0.001 0.001"/>
+    </geometry>
+  </collision>
+</link>
+<link name="suspension_front_right_1">
   <inertial>
     <origin xyz="0.0 -0.4032961129921663 0.0" rpy="0 0 0"/>
@@ -33,5 +33,5 @@
     <origin xyz="-1.925 -0.625 0.45" rpy="0 0 0"/>
     <geometry>
-      <mesh filename="file://$(find car_description)/meshes/suspension_back_left_1.stl" scale="0.001 0.001 0.001"/>
+      <mesh filename="file://$(find car)/meshes/suspension_front_right_1.stl" scale="0.001 0.001 0.001"/>
     </geometry>
     <material name="silver"/>
@@ -40,9 +40,9 @@
     <origin xyz="-1.925 -0.625 0.45" rpy="0 0 0"/>
     <geometry>
-      <mesh filename="file://$(find car_description)/meshes/suspension_back_left_1.stl" scale="0.001 0.001 0.001"/>
-    </geometry>
-  </collision>
-</link>
-<link name="suspension_back_right__1">
+      <mesh filename="file://$(find car)/meshes/suspension_front_right_1.stl" scale="0.001 0.001 0.001"/>
+    </geometry>
+  </collision>
+</link>
+<link name="suspension_front_left__1">
   <inertial>
     <origin xyz="-2.220446049250313e-16 0.40329611299216594 0.0" rpy="0 0 0"/>
@@ -53,5 +53,5 @@
     <origin xyz="-1.925 -0.875 0.45" rpy="0 0 0"/>
     <geometry>
-      <mesh filename="file://$(find car_description)/meshes/suspension_back_right__1.stl" scale="0.001 0.001 0.001"/>
+      <mesh filename="file://$(find car)/meshes/suspension_front_left__1.stl" scale="0.001 0.001 0.001"/>
     </geometry>
     <material name="silver"/>
@@ -60,9 +60,9 @@
     <origin xyz="-1.925 -0.875 0.45" rpy="0 0 0"/>
     <geometry>
-      <mesh filename="file://$(find car_description)/meshes/suspension_back_right__1.stl" scale="0.001 0.001 0.001"/>
-    </geometry>
-  </collision>
-</link>
-<link name="suspension_front_left_1">
+      <mesh filename="file://$(find car)/meshes/suspension_front_left__1.stl" scale="0.001 0.001 0.001"/>
+    </geometry>
+  </collision>
+</link>
+<link name="suspension_back_right_1">
   <inertial>
     <origin xyz="0.0 -0.4032961129921663 0.0" rpy="0 0 0"/>
@@ -73,5 +73,5 @@
     <origin xyz="-0.575 -0.625 0.45" rpy="0 0 0"/>
     <geometry>
-      <mesh filename="file://$(find car_description)/meshes/suspension_front_left_1.stl" scale="0.001 0.001 0.001"/>
+      <mesh filename="file://$(find car)/meshes/suspension_back_right_1.stl" scale="0.001 0.001 0.001"/>
     </geometry>
     <material name="silver"/>
@@ -80,9 +80,9 @@
     <origin xyz="-0.575 -0.625 0.45" rpy="0 0 0"/>
     <geometry>
-      <mesh filename="file://$(find car_description)/meshes/suspension_front_left_1.stl" scale="0.001 0.001 0.001"/>
-    </geometry>
-  </collision>
-</link>
-<link name="suspension_front_right_1">
+      <mesh filename="file://$(find car)/meshes/suspension_back_right_1.stl" scale="0.001 0.001 0.001"/>
+    </geometry>
+  </collision>
+</link>
+<link name="suspension_back_left_1">
   <inertial>
     <origin xyz="1.1102230246251565e-16 0.40329611299216617 0.0" rpy="0 0 0"/>
@@ -93,5 +93,5 @@
     <origin xyz="-0.575 -0.875 0.45" rpy="0 0 0"/>
     <geometry>
-      <mesh filename="file://$(find car_description)/meshes/suspension_front_right_1.stl" scale="0.001 0.001 0.001"/>
+      <mesh filename="file://$(find car)/meshes/suspension_back_left_1.stl" scale="0.001 0.001 0.001"/>
     </geometry>
     <material name="silver"/>
@@ -100,5 +100,5 @@
     <origin xyz="-0.575 -0.875 0.45" rpy="0 0 0"/>
     <geometry>
-      <mesh filename="file://$(find car_description)/meshes/suspension_front_right_1.stl" scale="0.001 0.001 0.001"/>
+      <mesh filename="file://$(find car)/meshes/suspension_back_left_1.stl" scale="0.001 0.001 0.001"/>
     </geometry>
   </collision>
@@ -113,5 +113,5 @@
     <origin xyz="-0.58 -1.75 0.45" rpy="0 0 0"/>
     <geometry>
-      <mesh filename="file://$(find car_description)/meshes/rim_back_left_1.stl" scale="0.001 0.001 0.001"/>
+      <mesh filename="file://$(find car)/meshes/rim_back_left_1.stl" scale="0.001 0.001 0.001"/>
     </geometry>
     <material name="silver"/>
@@ -120,5 +120,5 @@
     <origin xyz="-0.58 -1.75 0.45" rpy="0 0 0"/>
     <geometry>
-      <mesh filename="file://$(find car_description)/meshes/rim_back_left_1.stl" scale="0.001 0.001 0.001"/>
+      <mesh filename="file://$(find car)/meshes/rim_back_left_1.stl" scale="0.001 0.001 0.001"/>
     </geometry>
   </collision>
@@ -133,5 +133,5 @@
     <origin xyz="-0.58 0.25 0.45" rpy="0 0 0"/>
     <geometry>
-      <mesh filename="file://$(find car_description)/meshes/rim_back_right_1.stl" scale="0.001 0.001 0.001"/>
+      <mesh filename="file://$(find car)/meshes/rim_back_right_1.stl" scale="0.001 0.001 0.001"/>
     </geometry>
     <material name="silver"/>
@@ -140,5 +140,5 @@
     <origin xyz="-0.58 0.25 0.45" rpy="0 0 0"/>
     <geometry>
-      <mesh filename="file://$(find car_description)/meshes/rim_back_right_1.stl" scale="0.001 0.001 0.001"/>
+      <mesh filename="file://$(find car)/meshes/rim_back_right_1.stl" scale="0.001 0.001 0.001"/>
     </geometry>
   </collision>
@@ -153,5 +153,5 @@
     <origin xyz="-1.925 0.25 0.45" rpy="0 0 0"/>
     <geometry>
-      <mesh filename="file://$(find car_description)/meshes/rim_front_right_1.stl" scale="0.001 0.001 0.001"/>
+      <mesh filename="file://$(find car)/meshes/rim_front_right_1.stl" scale="0.001 0.001 0.001"/>
     </geometry>
     <material name="silver"/>
@@ -160,5 +160,5 @@
     <origin xyz="-1.925 0.25 0.45" rpy="0 0 0"/>
     <geometry>
-      <mesh filename="file://$(find car_description)/meshes/rim_front_right_1.stl" scale="0.001 0.001 0.001"/>
+      <mesh filename="file://$(find car)/meshes/rim_front_right_1.stl" scale="0.001 0.001 0.001"/>
     </geometry>
   </collision>
@@ -173,5 +173,5 @@
     <origin xyz="-1.925 -1.75 0.45" rpy="0 0 0"/>
     <geometry>
-      <mesh filename="file://$(find car_description)/meshes/rim_front_left_1.stl" scale="0.001 0.001 0.001"/>
+      <mesh filename="file://$(find car)/meshes/rim_front_left_1.stl" scale="0.001 0.001 0.001"/>
     </geometry>
     <material name="silver"/>
@@ -180,5 +180,5 @@
     <origin xyz="-1.925 -1.75 0.45" rpy="0 0 0"/>
     <geometry>
-      <mesh filename="file://$(find car_description)/meshes/rim_front_left_1.stl" scale="0.001 0.001 0.001"/>
+      <mesh filename="file://$(find car)/meshes/rim_front_left_1.stl" scale="0.001 0.001 0.001"/>
     </geometry>
   </collision>
@@ -193,5 +193,5 @@
     <origin xyz="-1.925 0.297622 0.45" rpy="0 0 0"/>
     <geometry>
-      <mesh filename="file://$(find car_description)/meshes/tire_front_right_1.stl" scale="0.001 0.001 0.001"/>
+      <mesh filename="file://$(find car)/meshes/tire_front_right_1.stl" scale="0.001 0.001 0.001"/>
     </geometry>
     <material name="silver"/>
@@ -200,5 +200,5 @@
     <origin xyz="-1.925 0.297622 0.45" rpy="0 0 0"/>
     <geometry>
-      <mesh filename="file://$(find car_description)/meshes/tire_front_right_1.stl" scale="0.001 0.001 0.001"/>
+      <mesh filename="file://$(find car)/meshes/tire_front_right_1.stl" scale="0.001 0.001 0.001"/>
     </geometry>
   </collision>
@@ -213,5 +213,5 @@
     <origin xyz="-0.58 0.297622 0.45" rpy="0 0 0"/>
     <geometry>
-      <mesh filename="file://$(find car_description)/meshes/tire_back_right_1.stl" scale="0.001 0.001 0.001"/>
+      <mesh filename="file://$(find car)/meshes/tire_back_right_1.stl" scale="0.001 0.001 0.001"/>
     </geometry>
     <material name="silver"/>
@@ -220,5 +220,5 @@
     <origin xyz="-0.58 0.297622 0.45" rpy="0 0 0"/>
     <geometry>
-      <mesh filename="file://$(find car_description)/meshes/tire_back_right_1.stl" scale="0.001 0.001 0.001"/>
+      <mesh filename="file://$(find car)/meshes/tire_back_right_1.stl" scale="0.001 0.001 0.001"/>
     </geometry>
   </collision>
@@ -233,5 +233,5 @@
     <origin xyz="-0.58 -1.797622 0.45" rpy="0 0 0"/>
     <geometry>
-      <mesh filename="file://$(find car_description)/meshes/tire_back_left_1.stl" scale="0.001 0.001 0.001"/>
+      <mesh filename="file://$(find car)/meshes/tire_back_left_1.stl" scale="0.001 0.001 0.001"/>
     </geometry>
     <material name="silver"/>
@@ -240,5 +240,5 @@
     <origin xyz="-0.58 -1.797622 0.45" rpy="0 0 0"/>
     <geometry>
-      <mesh filename="file://$(find car_description)/meshes/tire_back_left_1.stl" scale="0.001 0.001 0.001"/>
+      <mesh filename="file://$(find car)/meshes/tire_back_left_1.stl" scale="0.001 0.001 0.001"/>
     </geometry>
   </collision>
@@ -253,5 +253,5 @@
     <origin xyz="-1.925 -1.797622 0.45" rpy="0 0 0"/>
     <geometry>
-      <mesh filename="file://$(find car_description)/meshes/tire_front_left_1.stl" scale="0.001 0.001 0.001"/>
+      <mesh filename="file://$(find car)/meshes/tire_front_left_1.stl" scale="0.001 0.001 0.001"/>
     </geometry>
     <material name="silver"/>
@@ -260,9 +260,9 @@
     <origin xyz="-1.925 -1.797622 0.45" rpy="0 0 0"/>
     <geometry>
-      <mesh filename="file://$(find car_description)/meshes/tire_front_left_1.stl" scale="0.001 0.001 0.001"/>
-    </geometry>
-  </collision>
-</link>
-<link name="direction_front_right_1">
+      <mesh filename="file://$(find car)/meshes/tire_front_left_1.stl" scale="0.001 0.001 0.001"/>
+    </geometry>
+  </collision>
+</link>
+<link name="direction_back_left_1">
   <inertial>
     <origin xyz="0.00201472265142022 0.07474229529205378 5.551115123125783e-17" rpy="0 0 0"/>
@@ -273,5 +273,5 @@
     <origin xyz="-0.575 -1.5875 0.45" rpy="0 0 0"/>
     <geometry>
-      <mesh filename="file://$(find car_description)/meshes/direction_front_right_1.stl" scale="0.001 0.001 0.001"/>
+      <mesh filename="file://$(find car)/meshes/direction_back_left_1.stl" scale="0.001 0.001 0.001"/>
     </geometry>
     <material name="silver"/>
@@ -280,9 +280,9 @@
     <origin xyz="-0.575 -1.5875 0.45" rpy="0 0 0"/>
     <geometry>
-      <mesh filename="file://$(find car_description)/meshes/direction_front_right_1.stl" scale="0.001 0.001 0.001"/>
-    </geometry>
-  </collision>
-</link>
-<link name="direction_front_left_1">
+      <mesh filename="file://$(find car)/meshes/direction_back_left_1.stl" scale="0.001 0.001 0.001"/>
+    </geometry>
+  </collision>
+</link>
+<link name="direction_back_right_1">
   <inertial>
     <origin xyz="0.002014722651420442 -0.07474229529205342 0.0" rpy="0 0 0"/>
@@ -293,5 +293,5 @@
     <origin xyz="-0.575 0.0875 0.45" rpy="0 0 0"/>
     <geometry>
-      <mesh filename="file://$(find car_description)/meshes/direction_front_left_1.stl" scale="0.001 0.001 0.001"/>
+      <mesh filename="file://$(find car)/meshes/direction_back_right_1.stl" scale="0.001 0.001 0.001"/>
     </geometry>
     <material name="silver"/>
@@ -300,9 +300,9 @@
     <origin xyz="-0.575 0.0875 0.45" rpy="0 0 0"/>
     <geometry>
-      <mesh filename="file://$(find car_description)/meshes/direction_front_left_1.stl" scale="0.001 0.001 0.001"/>
-    </geometry>
-  </collision>
-</link>
-<link name="direction_back_left_1">
+      <mesh filename="file://$(find car)/meshes/direction_back_right_1.stl" scale="0.001 0.001 0.001"/>
+    </geometry>
+  </collision>
+</link>
+<link name="direction_front_right_1">
   <inertial>
     <origin xyz="-2.220446049250313e-16 -0.07474229529205345 0.0" rpy="0 0 0"/>
@@ -313,5 +313,5 @@
     <origin xyz="-1.925 0.0875 0.45" rpy="0 0 0"/>
     <geometry>
-      <mesh filename="file://$(find car_description)/meshes/direction_back_left_1.stl" scale="0.001 0.001 0.001"/>
+      <mesh filename="file://$(find car)/meshes/direction_front_right_1.stl" scale="0.001 0.001 0.001"/>
     </geometry>
     <material name="silver"/>
@@ -320,9 +320,9 @@
     <origin xyz="-1.925 0.0875 0.45" rpy="0 0 0"/>
     <geometry>
-      <mesh filename="file://$(find car_description)/meshes/direction_back_left_1.stl" scale="0.001 0.001 0.001"/>
-    </geometry>
-  </collision>
-</link>
-<link name="direction_back_right_1">
+      <mesh filename="file://$(find car)/meshes/direction_front_right_1.stl" scale="0.001 0.001 0.001"/>
+    </geometry>
+  </collision>
+</link>
+<link name="direction_front_left_1">
   <inertial>
     <origin xyz="2.220446049250313e-16 0.07474229529205334 5.551115123125783e-17" rpy="0 0 0"/>
@@ -333,5 +333,5 @@
     <origin xyz="-1.925 -1.5875 0.45" rpy="0 0 0"/>
     <geometry>
-      <mesh filename="file://$(find car_description)/meshes/direction_back_right_1.stl" scale="0.001 0.001 0.001"/>
+      <mesh filename="file://$(find car)/meshes/direction_front_left_1.stl" scale="0.001 0.001 0.001"/>
     </geometry>
     <material name="silver"/>
@@ -340,65 +340,65 @@
     <origin xyz="-1.925 -1.5875 0.45" rpy="0 0 0"/>
     <geometry>
-      <mesh filename="file://$(find car_description)/meshes/direction_back_right_1.stl" scale="0.001 0.001 0.001"/>
-    </geometry>
-  </collision>
-</link>
-<link name="Lidar_1">
-  <inertial>
-    <origin xyz="-6.661338147750939e-16 -1.1102230246251565e-16 0.04999999999999993" rpy="0 0 0"/>
+      <mesh filename="file://$(find car)/meshes/direction_front_left_1.stl" scale="0.001 0.001 0.001"/>
+    </geometry>
+  </collision>
+</link>
+<link name="chasis_1">
+  <inertial>
+    <origin xyz="0.09238270773822022 -1.1102230246251565e-16 0.5327884318036318" rpy="0 0 0"/>
+    <mass value="14235.910080029777"/>
+    <inertia ixx="3772.896581" iyy="5428.125259" izz="8145.031104" ixy="0.0" iyz="-0.0" ixz="-431.237028"/>
+  </inertial>
+  <visual>
+    <origin xyz="-1.25 -0.75 0.4" rpy="0 0 0"/>
+    <geometry>
+      <mesh filename="file://$(find car)/meshes/chasis_1.stl" scale="0.001 0.001 0.001"/>
+    </geometry>
+    <material name="silver"/>
+  </visual>
+  <collision>
+    <origin xyz="-1.25 -0.75 0.4" rpy="0 0 0"/>
+    <geometry>
+      <mesh filename="file://$(find car)/meshes/chasis_1.stl" scale="0.001 0.001 0.001"/>
+    </geometry>
+  </collision>
+</link>
+<link name="Component24_1">
+  <inertial>
+    <origin xyz="-6.661338147750939e-16 1.1102230246251565e-16 0.050000000000000266" rpy="0 0 0"/>
     <mass value="24.661502330679863"/>
-    <inertia ixx="0.082205" iyy="0.082205" izz="0.123308" ixy="-0.0" iyz="0.0" ixz="-0.0"/>
-  </inertial>
-  <visual>
-    <origin xyz="-1.85 -0.75 -0.7" rpy="0 0 0"/>
-    <geometry>
-      <mesh filename="file://$(find car_description)/meshes/Lidar_1.stl" scale="0.001 0.001 0.001"/>
-    </geometry>
-    <material name="silver"/>
-  </visual>
-  <collision>
-    <origin xyz="-1.85 -0.75 -0.7" rpy="0 0 0"/>
-    <geometry>
-      <mesh filename="file://$(find car_description)/meshes/Lidar_1.stl" scale="0.001 0.001 0.001"/>
-    </geometry>
-  </collision>
-</link>
-<link name="Camara_1">
-  <inertial>
-    <origin xyz="-0.004642640365980721 0.0 -0.0018567286993164678" rpy="0 0 0"/>
-    <mass value="3.1890625000000425"/>
-    <inertia ixx="0.031654" iyy="0.004179" izz="0.028666" ixy="0.0" iyz="0.0" ixz="0.001423"/>
-  </inertial>
-  <visual>
-    <origin xyz="-2.162084 -0.7625 -0.447483" rpy="0 0 0"/>
-    <geometry>
-      <mesh filename="file://$(find car_description)/meshes/Camara_1.stl" scale="0.001 0.001 0.001"/>
-    </geometry>
-    <material name="silver"/>
-  </visual>
-  <collision>
-    <origin xyz="-2.162084 -0.7625 -0.447483" rpy="0 0 0"/>
-    <geometry>
-      <mesh filename="file://$(find car_description)/meshes/Camara_1.stl" scale="0.001 0.001 0.001"/>
-    </geometry>
-  </collision>
-</link>
-<link name="chasis_1">
-  <inertial>
-    <origin xyz="0.09270352913138602 2.798168493578501e-07 0.5332144331317273" rpy="0 0 0"/>
-    <mass value="14246.204737445123"/>
-    <inertia ixx="3776.349491" iyy="5433.367868" izz="8146.852846" ixy="-0.003264" iyz="-0.001252" ixz="-434.117699"/>
-  </inertial>
-  <visual>
-    <origin xyz="-1.25 -0.75 0.4" rpy="0 0 0"/>
-    <geometry>
-      <mesh filename="file://$(find car_description)/meshes/chasis_1.stl" scale="0.001 0.001 0.001"/>
-    </geometry>
-    <material name="silver"/>
-  </visual>
-  <collision>
-    <origin xyz="-1.25 -0.75 0.4" rpy="0 0 0"/>
-    <geometry>
-      <mesh filename="file://$(find car_description)/meshes/chasis_1.stl" scale="0.001 0.001 0.001"/>
+    <inertia ixx="0.082205" iyy="0.082205" izz="0.123308" ixy="0.0" iyz="-0.0" ixz="0.0"/>
+  </inertial>
+  <visual>
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
Commit message: model only lidar

File: workspace/src/car_python/urdf/car.xacro (robot description, xacro)
@@ -364,5 +364,5 @@
   </collision>
 </link>
-<link name="Component24_1">
+<link name="Lidar_1">
   <inertial>
     <origin xyz="-6.661338147750939e-16 1.1102230246251565e-16 0.050000000000000266" rpy="0 0 0"/>
@@ -373,5 +373,5 @@
     <origin xyz="-1.85 -0.75 -0.65" rpy="0 0 0"/>
     <geometry>
-      <mesh filename="file://$(find car)/meshes/Component24_1.stl" scale="0.001 0.001 0.001"/>
+      <mesh filename="file://$(find car)/meshes/Lidar_1.stl" scale="0.001 0.001 0.001"/>
     </geometry>
     <material name="silver"/>
@@ -380,25 +380,5 @@
     <origin xyz="-1.85 -0.75 -0.65" rpy="0 0 0"/>
     <geometry>
-      <mesh filename="file://$(find car)/meshes/Component24_1.stl" scale="0.001 0.001 0.001"/>
-    </geometry>
-  </collision>
-</link>
-<link name="Component25_1">
-  <inertial>
-    <origin xyz="0.004642800215263865 0.0 0.0018567355153457643" rpy="0 0 0"/>
-    <mass value="2.3549999999999622"/>
-    <inertia ixx="0.019357" iyy="0.001982" izz="0.01795" ixy="-0.0" iyz="-0.0" ixz="0.00067"/>
-  </inertial>
-  <visual>
-    <origin xyz="-2.175082 -0.75 -0.43922" rpy="0 0 0"/>
-    <geometry>
-      <mesh filename="file://$(find car)/meshes/Component25_1.stl" scale="0.001 0.001 0.001"/>
-    </geometry>
-    <material name="silver"/>
-  </visual>
-  <collision>
-    <origin xyz="-2.175082 -0.75 -0.43922" rpy="0 0 0"/>
-    <geometry>
-      <mesh filename="file://$(find car)/meshes/Component25_1.stl" scale="0.001 0.001 0.001"/>
+      <mesh filename="file://$(find car)/meshes/Lidar_1.stl" scale="0.001 0.001 0.001"/>
     </geometry>
   </collision>
@@ -509,13 +489,8 @@
   <child link="chasis_1"/>
 </joint>
-<joint name="Rigid 22" type="fixed">
+<joint name="Rigid 24" type="fixed">
   <origin xyz="0.6 0.0 1.05" rpy="0 0 0"/>
   <parent link="chasis_1"/>
-  <child link="Component24_1"/>
-</joint>
-<joint name="Rigid 23" type="fixed">
-  <origin xyz="0.925082 0.0 0.83922" rpy="0 0 0"/>
-  <parent link="chasis_1"/>
-  <child link="Component25_1"/>
+  <child link="Lidar_1"/>
 </joint>
 </robot>

Commit message: test model

File: workspace/src/car_python/urdf/car.xacro (robot description, xacro)
@@ -384,4 +384,24 @@
   </collision>
 </link>
+<link name="camara_1">
+  <inertial>
+    <origin xyz="0.004642800215263865 0.0 0.0018567355153457643" rpy="0 0 0"/>
+    <mass value="2.3549999999999622"/>
+    <inertia ixx="0.019357" iyy="0.001982" izz="0.01795" ixy="-0.0" iyz="-0.0" ixz="0.00067"/>
+  </inertial>
+  <visual>
+    <origin xyz="-2.175082 -0.75 -0.43922" rpy="0 0 0"/>
+    <geometry>
+      <mesh filename="file://$(find car)/meshes/camara_1.stl" scale="0.001 0.001 0.001"/>
+    </geometry>
+    <material name="silver"/>
+  </visual>
+  <collision>
+    <origin xyz="-2.175082 -0.75 -0.43922" rpy="0 0 0"/>
+    <geometry>
+      <mesh filename="file://$(find car)/meshes/camara_1.stl" scale="0.001 0.001 0.001"/>
+    </geometry>
+  </collision>
+</link>
 <joint name="Revolute 1" type="revolute">
   <origin xyz="1.925 0.625 -0.45" rpy="0 0 0"/>
@@ -494,3 +514,8 @@
   <child link="Lidar_1"/>
 </joint>
+<joint name="Rigid 25" type="fixed">
+  <origin xyz="0.925082 0.0 0.83922" rpy="0 0 0"/>
+  <parent link="chasis_1"/>
+  <child link="camara_1"/>
+</joint>
 </robot>
