Commit message: works map , but needed to fix the map, for now is using the scan stamp, need to add the true odometry and fix the map dont move with the model, next its 3d

File: workspace_full_conected/install/car/share/car/urdf/camara.plugin.xacro (robot description, xacro)
@@ -9,6 +9,6 @@
                 <horizontal_fov>2</horizontal_fov>
                 <image>
-                    <width>640</width>
-                    <height>480</height>
+                    <width>1920</width>
+                    <height>1080</height>
                     <format>R8G8B8</format>
                 </image>
@@ -19,5 +19,5 @@
             </camera>
             <plugin name="depth_camera_controller" filename="libgazebo_ros_camera.so">
-                <frame_name>camera_optical_frame</frame_name>
+                <frame_name>odom</frame_name>
             </plugin>
         </sensor>

File: workspace_full_conected/install/car/share/car/urdf/car.xacro (robot description, xacro)
@@ -5,5 +5,5 @@
 <xacro:include filename="$(find car)/urdf/car.gazebo" />
 <xacro:include filename="$(find car)/urdf/camara.plugin.xacro" />
-<!-- <xacro:include filename="$(find car)/urdf/lidar.plugin.xacro" /> -->
+<xacro:include filename="$(find car)/urdf/lidar.plugin.xacro" />
 <link name="base_link">
   <inertial>
@@ -527,4 +527,14 @@
   </plugin>
 </gazebo>
+<!-- <gazebo>
+  <plugin name="odometryPlugin" filename="libodometry_plugin.so">
+    <left_front_wheel_joint>Revolute 17</left_front_wheel_joint>
+    <right_front_wheel_joint>Revolute 16</right_front_wheel_joint>
+    <left_back_wheel_joint>Revolute 5</left_back_wheel_joint>
+    <right_back_wheel_joint>Revolute 6</right_back_wheel_joint>
+    <left_front_speed_wheel_joint>Revolute 8</left_front_speed_wheel_joint>
+    <right_front_speed_wheel_joint>Revolute 7</right_front_speed_wheel_joint>
+  </plugin>
+</gazebo> -->
 <link name="camera_optical_frame">
 </link>
@@ -535,5 +545,13 @@
   <origin xyz="0 0 0" rpy="-1.5708 0 -1.5708"/>
 </joint>
-<gazebo>
+<link name="base_footprint">
+</link>
+<joint name="base_footprint" type="fixed">
+  <parent link="base_link"/>
+  <child link="base_footprint"/>
+  <!-- Ajusta rpy para alinear el frame óptico -->
+  <origin xyz="0 0 0" rpy="0 0 0"/>
+</joint>
+<!-- <gazebo>
   <plugin name="imu_controller" filename="libhector_gazebo_ros_imu.so">
   <robotNamespace>car</robotNamespace>
@@ -563,4 +581,4 @@
   <drift>0.0001 0.0001 0.0001</drift>
   </plugin>
-</gazebo>
+</gazebo> -->
 </robot>

File: workspace_full_conected/install/car/share/car/urdf/lidar.plugin.xacro (robot description, xacro)
@@ -3,25 +3,20 @@
 <!-- Laser sensor plugin -->
   <gazebo reference="Lidar">
-    <sensor type="gpu_ray" name="laser_sensor">
+    <sensor type="ray" name="laser">
       <pose>0 0 0 0 0 0</pose>
-      <visualize>false</visualize>
-      <update_rate>30.0</update_rate>
+      <visualize>true</visualize>
+      <update_rate>10.0</update_rate>
       <ray>
         <scan>
-          <horizontal>
+        <horizontal>
             <samples>360</samples>
             <resolution>1</resolution>
             <min_angle>-3.14</min_angle> <!-- -180 degrees -->
             <max_angle>3.14</max_angle>  <!-- 180 degrees -->
-          </horizontal>
-          <vertical>
-            <samples>360</samples> <!-- Número de "líneas" verticales que va a capturar -->
-            <min_angle>-0.3</min_angle> <!-- 45 degrees -->
-            <max_angle>0.3</max_angle>  <!-- 45 degress -->
-          </vertical>
+        </horizontal>
         </scan>
         <range>
-          <min>0.1</min>
-          <max>10.0</max>
+          <min>0.3</min>
+          <max>12.0</max>
           <resolution>0.01</resolution>
         </range>
@@ -32,8 +27,13 @@
         </noise>
       </ray>
-      <plugin name="gazebo_ros_laser" filename="libgazebo_ros_ray_sensor.so">
-        <topicName>/scan</topicName>
-        <frameName>Lidar</frameName>
-        <!-- <output_type>sensor_msgs/PointCloud2</output_type> -->
+      <plugin name="laser_controller" filename="libgazebo_ros_ray_sensor.so">
+        <ros>
+          <argument>use_sim_time:=true</argument>
+          <argument>~/out:=/scan</argument>
+        </ros>
+        <frame_name>base_link</frame_name>
+        <fixed_frame>odom</fixed_frame>
+        <publish_tf>true</publish_tf>
+        <output_type>sensor_msgs/LaserScan</output_type>
       </plugin>
     </sensor>

Commit message: work all the map and plugins

File: workspace_full_conected/install/car/share/car/urdf/camara.plugin.xacro (robot description, xacro)
@@ -5,10 +5,10 @@
             <pose>0 0 0 0 0 0</pose>
             <visualize>true</visualize>
-            <update_rate>30.0</update_rate>
+            <update_rate>100.0</update_rate>
             <camera>
                 <horizontal_fov>2</horizontal_fov>
                 <image>
-                    <width>1920</width>
-                    <height>1080</height>
+                    <width>640</width>
+                    <height>480</height>
                     <format>R8G8B8</format>
                 </image>
@@ -19,5 +19,9 @@
             </camera>
             <plugin name="depth_camera_controller" filename="libgazebo_ros_camera.so">
-                <frame_name>odom</frame_name>
+                        <ros>
+                            <argument>use_sim_time:=true</argument>
+                        </ros>
+                <frame_name>camera_optical_frame</frame_name>
+                <publish_tf>true</publish_tf>
             </plugin>
         </sensor>

File: workspace_full_conected/install/car/share/car/urdf/car.xacro (robot description, xacro)
@@ -517,5 +517,5 @@
   <child link="Camara"/>
 </joint>
-<gazebo>
+<!-- <gazebo>
   <plugin name="ControlPlugin" filename="libcontrol_plugin.so">
     <left_front_wheel_joint>front_left_wheel_joint</left_front_wheel_joint>
@@ -524,31 +524,12 @@
     <right_back_wheel_joint>back_right_wheel_joint</right_back_wheel_joint>
   </plugin>
-</gazebo>
-<gazebo>
-    <plugin name="joint_state_publisher" filename="libgazebo_ros_joint_state_publisher.so">
-      <ros>
-        <namespace>car</namespace>
-        <remapping>joint_states:=/joint_states</remapping>
-      </ros>
-      <update_rate>50</update_rate>
-    </plugin>
-  </gazebo>
-<!-- <gazebo>
-  <plugin name="odometryPlugin" filename="libodometry_plugin.so">
-    <left_front_wheel_joint>Revolute 17</left_front_wheel_joint>
-    <right_front_wheel_joint>Revolute 16</right_front_wheel_joint>
-    <left_back_wheel_joint>Revolute 5</left_back_wheel_joint>
-    <right_back_wheel_joint>Revolute 6</right_back_wheel_joint>
-    <left_front_speed_wheel_joint>Revolute 8</left_front_speed_wheel_joint>
-    <right_front_speed_wheel_joint>Revolute 7</right_front_speed_wheel_joint>
-  </plugin>
 </gazebo> -->
 <link name="camera_optical_frame">
 </link>
 <joint name="camera_optical_joint" type="fixed">
-  <parent link="Camara"/>
-  <child link="camera_optical_frame"/>
-  <!-- Ajusta rpy para alinear el frame óptico -->
-  <origin xyz="0 0 0" rpy="-1.5708 0 -1.5708"/>
+<parent link="Camara"/>
+<child link="camera_optical_frame"/>
+<!-- Ajusta rpy para alinear el frame óptico -->
+<origin xyz="0 0 0" rpy="-1.5708 0 -1.5708"/>
 </joint>
 <link name="base_footprint">
@@ -560,5 +541,13 @@
   <origin xyz="0 0 0" rpy="0 0 0"/>
 </joint>
-<gazebo>
+<link name="lidar_footprint">
+</link>
+<joint name="lidar_footprint" type="fixed">
+  <parent link="Lidar"/>
+  <child link="lidar_footprint"/>
+  <!-- Ajusta rpy para alinear el frame óptico -->
+  <origin xyz="0 0 0" rpy="0 0 0"/>
+</joint>
+ <gazebo>
   <plugin name="imu_controller" filename="libhector_gazebo_ros_imu.so">
   <robotNamespace>car</robotNamespace>
@@ -577,5 +566,5 @@
   <plugin name="gps_controller" filename="libhector_gazebo_ros_gps.so">
   <robotNamespace>car</robotNamespace>
-  <updateRate>40</updateRate>
+  <updateRate>50</updateRate>
   <bodyName>base_link</bodyName>
   <frameId>base_link</frameId>
@@ -589,3 +578,34 @@
   </plugin>
 </gazebo>
+<gazebo>
+  <plugin name="gazebo_ros_diff_drive_multi_wheel" filename="libdrive_plugin.so">
+     <robotNamespace>/car</robotNamespace>
+      <leftJoints>front_left_wheel_joint back_left_wheel_joint</leftJoints>
+      <rightJoints>front_right_wheel_joint back_right_wheel_joint</rightJoints>
+      <wheelSeparation>0.34</wheelSeparation>
+      <wheelDiameter>0.15</wheelDiameter>
+      <torque>5.0</torque>
+      <commandTopic>cmd_vel</commandTopic>
+      <odometryTopic>odom</odometryTopic>
+      <odometryFrame>odom</odometryFrame>
+      <robotBaseFrame>base_link</robotBaseFrame>
+      <updateRate>100</updateRate>
+      <publishOdometryTf>true</publishOdometryTf>
+      <publishOdometryMsg>true</publishOdometryMsg>
+      <!-- Parámetros para la transformación del Lidar -->
+      <lidarLink>lidar_footprint</lidarLink>
+      <lidarPose>
+        <x>0.6</x>
+        <y>0.0</y>
+        <z>1.05</z>
+        <!-- Si se requiere orientación, se pueden incluir roll, pitch y yaw -->
+      </lidarPose>
+    </plugin>
+  </gazebo>
+<gazebo>
+  <plugin name="joint_state_publisher_plugin" filename="libjoints_plugin.so">
+    <robotNamespace>car</robotNamespace>
+    <updateRate>50.0</updateRate>
+  </plugin>
+</gazebo>
 </robot>

File: workspace_full_conected/install/car/share/car/urdf/lidar.plugin.xacro (robot description, xacro)
@@ -1,18 +1,23 @@
 <?xml version="1.0" ?>
 <robot>
-<!-- Laser sensor plugin -->
+  <!-- LiDAR 3D con gpu_ray -->
   <gazebo reference="Lidar">
-    <sensor type="ray" name="laser">
+    <sensor type="gpu_ray" name="Lidar">
       <pose>0 0 0 0 0 0</pose>
-      <visualize>true</visualize>
+      <visualize>false</visualize>
       <update_rate>10.0</update_rate>
       <ray>
         <scan>
-        <horizontal>
+          <horizontal>
             <samples>360</samples>
-            <resolution>1</resolution>
-            <min_angle>-3.14</min_angle> <!-- -180 degrees -->
-            <max_angle>3.14</max_angle>  <!-- 180 degrees -->
-        </horizontal>
+            <min_angle>-3.14</min_angle>
+            <max_angle>3.14</max_angle>
+          </horizontal>
+          <vertical>
+            <!-- Define un barrido vertical; ajusta samples y ángulos según el FOV deseado -->
+            <samples>16</samples>
+            <min_angle>-0.2618</min_angle>  <!-- -15° -->
+            <max_angle>0.2618</max_angle>    <!-- 15° -->
+          </vertical>
         </scan>
         <range>
@@ -27,13 +32,13 @@
         </noise>
       </ray>
-      <plugin name="laser_controller" filename="libgazebo_ros_ray_sensor.so">
+      <plugin name="lidar_controller" filename="libgazebo_ros_ray_sensor.so">
         <ros>
           <argument>use_sim_time:=true</argument>
-          <argument>~/out:=/scan</argument>
+          <!-- Publica directamente en un topic; si deseas trabajar con nubes de puntos, puedes publicar PointCloud2 -->
+          <argument>~/out:=/scan_cloud</argument>
         </ros>
-        <frame_name>base_link</frame_name>
-        <fixed_frame>odom</fixed_frame>
-        <publish_tf>true</publish_tf>
-        <output_type>sensor_msgs/LaserScan</output_type>
+        <frame_name>Lidar</frame_name>
+        <!-- Especifica que el output es PointCloud2 -->
+        <output_type>sensor_msgs/PointCloud2</output_type>
       </plugin>
     </sensor>
