Commit message: keep working on it

File: workspace_full_conected/install/car/share/car/urdf/car.xacro (robot description, xacro)
@@ -434,5 +434,5 @@
   <limit upper="0.087266" lower="-0.174533" effort="100" velocity="100"/>
 </joint>
-<joint name="Revolute 5" type="continuous">
+<joint name="back_left_wheel_joint" type="continuous">
   <origin xyz="0.005 0.1625 0.0" rpy="0 0 0"/>
   <parent link="direction_back_left_1"/>
@@ -440,5 +440,5 @@
   <axis xyz="0.0 1.0 0.0"/>
 </joint>
-<joint name="Revolute 6" type="continuous">
+<joint name="back_right_wheel_joint" type="continuous">
   <origin xyz="0.005 -0.1625 0.0" rpy="0 0 0"/>
   <parent link="direction_back_right_1"/>
@@ -446,5 +446,5 @@
   <axis xyz="0.0 -1.0 0.0"/>
 </joint>
-<joint name="Revolute 7" type="continuous">
+<joint name="front_right_wheel_joint" type="continuous">
   <origin xyz="0.0 -0.1625 0.0" rpy="0 0 0"/>
   <parent link="direction_front_right_1"/>
@@ -452,5 +452,5 @@
   <axis xyz="0.0 -1.0 0.0"/>
 </joint>
-<joint name="Revolute 8" type="continuous">
+<joint name="front_left_wheel_joint" type="continuous">
   <origin xyz="0.0 0.1625 0.0" rpy="0 0 0"/>
   <parent link="direction_front_left_1"/>
@@ -488,5 +488,5 @@
   <child link="direction_back_right_1"/>
 </joint>
-<joint name="Revolute 16" type="revolute">
+<joint name="Revolute 16" type="fixed">
   <origin xyz="0.0 -0.7125 0.0" rpy="0 0 0"/>
   <parent link="suspension_front_right_1"/>
@@ -495,5 +495,5 @@
   <limit upper="0.523599" lower="-0.523599" effort="100" velocity="100"/>
 </joint>
-<joint name="Revolute 17" type="revolute">
+<joint name="Revolute 17" type="fixed">
   <origin xyz="0.0 0.7125 0.0" rpy="0 0 0"/>
   <parent link="suspension_front_left__1"/>
@@ -519,12 +519,19 @@
 <gazebo>
   <plugin name="ControlPlugin" filename="libcontrol_plugin.so">
-    <left_front_wheel_joint>Revolute 17</left_front_wheel_joint>
-    <right_front_wheel_joint>Revolute 16</right_front_wheel_joint>
-    <left_back_wheel_joint>Revolute 5</left_back_wheel_joint>
-    <right_back_wheel_joint>Revolute 6</right_back_wheel_joint>
-    <left_front_speed_wheel_joint>Revolute 8</left_front_speed_wheel_joint>
-    <right_front_speed_wheel_joint>Revolute 7</right_front_speed_wheel_joint>
+    <left_front_wheel_joint>front_left_wheel_joint</left_front_wheel_joint>
+    <right_front_wheel_joint>front_right_wheel_joint</right_front_wheel_joint>
+    <left_back_wheel_joint>back_left_wheel_joint</left_back_wheel_joint>
+    <right_back_wheel_joint>back_right_wheel_joint</right_back_wheel_joint>
   </plugin>
 </gazebo>
+<gazebo>
+    <plugin name="joint_state_publisher" filename="libgazebo_ros_joint_state_publisher.so">
+      <ros>
+        <namespace>car</namespace>
+        <remapping>joint_states:=/joint_states</remapping>
+      </ros>
+      <update_rate>50</update_rate>
+    </plugin>
+  </gazebo>
 <!-- <gazebo>
   <plugin name="odometryPlugin" filename="libodometry_plugin.so">
@@ -553,5 +560,5 @@
   <origin xyz="0 0 0" rpy="0 0 0"/>
 </joint>
-<!-- <gazebo>
+<gazebo>
   <plugin name="imu_controller" filename="libhector_gazebo_ros_imu.so">
   <robotNamespace>car</robotNamespace>
@@ -581,4 +588,4 @@
   <drift>0.0001 0.0001 0.0001</drift>
   </plugin>
-</gazebo> -->
+</gazebo>
 </robot>

Commit message: time to train

File: workspace_full_conected/install/car/share/car/urdf/car.xacro (robot description, xacro)
@@ -8,19 +8,119 @@
 <link name="base_link">
   <inertial>
+    <origin xyz="0.0 0.0 -5.8299495211720805e-18" rpy="0 0 0"/>
+    <mass value="195.94086385796686"/>
+    <inertia ixx="0.825102" iyy="42.139945" izz="42.62574" ixy="0.0" iyz="-0.0" ixz="0.0"/>
+  </inertial>
+  <visual>
     <origin xyz="0 0 0" rpy="0 0 0"/>
-    <mass value="195.94086385796686"/>
-    <inertia ixx="0.825102" iyy="42.139945" izz="42.62574" ixy="-0.0" iyz="0.0" ixz="0.0"/>
-  </inertial>
-  <visual>
+    <geometry>
+      <mesh filename="file://$(find car)/meshes/base_link.stl" scale="0.001 0.001 0.001"/>
+    </geometry>
+    <material name="silver"/>
+  </visual>
+  <collision>
     <origin xyz="0 0 0" rpy="0 0 0"/>
     <geometry>
       <mesh filename="file://$(find car)/meshes/base_link.stl" scale="0.001 0.001 0.001"/>
     </geometry>
-    <material name="silver"/>
-  </visual>
-  <collision>
-    <origin xyz="0 0 0" rpy="0 0 0"/>
-    <geometry>
-      <mesh filename="file://$(find car)/meshes/base_link.stl" scale="0.001 0.001 0.001"/>
+  </collision>
+</link>
+<link name="chasis_1">
+  <inertial>
+    <origin xyz="0.09238270773822028 0.0 0.5327884318036319" rpy="0 0 0"/>
+    <mass value="14235.910080029777"/>
+    <inertia ixx="3772.896581" iyy="5428.125259" izz="8145.031104" ixy="0.0" iyz="0.0" ixz="-431.237028"/>
+  </inertial>
+  <visual>
+    <origin xyz="-0.0 -0.0 -0.05" rpy="0 0 0"/>
+    <geometry>
+      <mesh filename="file://$(find car)/meshes/chasis_1.stl" scale="0.001 0.001 0.001"/>
+    </geometry>
+    <material name="silver"/>
+  </visual>
+  <collision>
+    <origin xyz="-0.0 -0.0 -0.05" rpy="0 0 0"/>
+    <geometry>
+      <mesh filename="file://$(find car)/meshes/chasis_1.stl" scale="0.001 0.001 0.001"/>
+    </geometry>
+  </collision>
+</link>
+<link name="suspension_front_left__1">
+  <inertial>
+    <origin xyz="-0.02499999999999991 0.4032961129921663 -1.7763568394002505e-17" rpy="0 0 0"/>
+    <mass value="33.21861256094089"/>
+    <inertia ixx="1.897101" iyy="0.053443" izz="1.887366" ixy="0.0" iyz="0.0" ixz="0.0"/>
+  </inertial>
+  <visual>
+    <origin xyz="-0.7 -0.125 -0.0" rpy="0 0 0"/>
+    <geometry>
+      <mesh filename="file://$(find car)/meshes/suspension_front_left__1.stl" scale="0.001 0.001 0.001"/>
+    </geometry>
+    <material name="silver"/>
+  </visual>
+  <collision>
+    <origin xyz="-0.7 -0.125 -0.0" rpy="0 0 0"/>
+    <geometry>
+      <mesh filename="file://$(find car)/meshes/suspension_front_left__1.stl" scale="0.001 0.001 0.001"/>
+    </geometry>
+  </collision>
+</link>
+<link name="direction_front_left_1">
+  <inertial>
+    <origin xyz="0.0 0.07474229529205356 -0.01999999999999999" rpy="0 0 0"/>
+    <mass value="11.38685889441971"/>
+    <inertia ixx="0.054235" iyy="0.024086" izz="0.067971" ixy="0.0" iyz="0.0" ixz="0.0"/>
+  </inertial>
+  <visual>
+    <origin xyz="-0.675 -0.8375 -0.02" rpy="0 0 0"/>
+    <geometry>
+      <mesh filename="file://$(find car)/meshes/direction_front_left_1.stl" scale="0.001 0.001 0.001"/>
+    </geometry>
+    <material name="silver"/>
+  </visual>
+  <collision>
+    <origin xyz="-0.675 -0.8375 -0.02" rpy="0 0 0"/>
+    <geometry>
+      <mesh filename="file://$(find car)/meshes/direction_front_left_1.stl" scale="0.001 0.001 0.001"/>
+    </geometry>
+  </collision>
+</link>
+<link name="rim_front_left_1">
+  <inertial>
+    <origin xyz="-8.236798832994552e-07 0.04445848581580858 3.411160743613806e-06" rpy="0 0 0"/>
+    <mass value="35.26167787649671"/>
+    <inertia ixx="0.833793" iyy="1.488731" izz="0.833793" ixy="-0.0" iyz="-3e-06" ixz="-1e-06"/>
+  </inertial>
+  <visual>
+    <origin xyz="-0.675 -1.0 -0.0" rpy="0 0 0"/>
+    <geometry>
+      <mesh filename="file://$(find car)/meshes/rim_front_left_1.stl" scale="0.001 0.001 0.001"/>
+    </geometry>
+    <material name="silver"/>
+  </visual>
+  <collision>
+    <origin xyz="-0.675 -1.0 -0.0" rpy="0 0 0"/>
+    <geometry>
+      <mesh filename="file://$(find car)/meshes/rim_front_left_1.stl" scale="0.001 0.001 0.001"/>
+    </geometry>
+  </collision>
+</link>
+<link name="tire_front_right_1">
+  <inertial>
+    <origin xyz="-2.55351295663786e-15 -1.8654241529247884e-07 1.4210854715202004e-16" rpy="0 0 0"/>
+    <mass value="72.81552294350315"/>
+    <inertia ixx="4.088543" iyy="7.430415" izz="4.088543" ixy="0.0" iyz="-0.0" ixz="-0.0"/>
+  </inertial>
+  <visual>
+    <origin xyz="-0.675 -1.047622 -0.0" rpy="0 0 0"/>
+    <geometry>
+      <mesh filename="file://$(find car)/meshes/tire_front_right_1.stl" scale="0.001 0.001 0.001"/>
+    </geometry>
+    <material name="silver"/>
+  </visual>
+  <collision>
+    <origin xyz="-0.675 -1.047622 -0.0" rpy="0 0 0"/>
+    <geometry>
+      <mesh filename="file://$(find car)/meshes/tire_front_right_1.stl" scale="0.001 0.001 0.001"/>
     </geometry>
   </collision>
@@ -28,10 +128,10 @@
 <link name="suspension_front_right_1">
   <inertial>
-    <origin xyz="0.0 -0.4032961129921663 0.0" rpy="0 0 0"/>
+    <origin xyz="-0.02499999999999991 -0.4032961129921663 0.0" rpy="0 0 0"/>
     <mass value="33.21861256094089"/>
     <inertia ixx="1.897101" iyy="0.053443" izz="1.887366" ixy="0.0" iyz="0.0" ixz="-0.0"/>
   </inertial>
   <visual>
-    <origin xyz="-1.925 -0.625 0.45" rpy="0 0 0"/>
+    <origin xyz="-0.7 0.125 -0.0" rpy="0 0 0"/>
     <geometry>
       <mesh filename="file://$(find car)/meshes/suspension_front_right_1.stl" scale="0.001 0.001 0.001"/>
@@ -40,5 +140,5 @@
   </visual>
   <collision>
-    <origin xyz="-1.925 -0.625 0.45" rpy="0 0 0"/>
+    <origin xyz="-0.7 0.125 -0.0" rpy="0 0 0"/>
     <geometry>
       <mesh filename="file://$(find car)/meshes/suspension_front_right_1.stl" scale="0.001 0.001 0.001"/>
@@ -46,52 +146,152 @@
   </collision>
 </link>
-<link name="suspension_front_left__1">
-  <inertial>
-    <origin xyz="-2.220446049250313e-16 0.40329611299216594 0.0" rpy="0 0 0"/>
+<link name="direction_front_right_1">
+  <inertial>
+    <origin xyz="-3.3306690738754696e-16 -0.07474229529205345 0.02" rpy="0 0 0"/>
+    <mass value="11.386858894419674"/>
+    <inertia ixx="0.054235" iyy="0.024086" izz="0.067971" ixy="0.0" iyz="0.0" ixz="0.0"/>
+  </inertial>
+  <visual>
+    <origin xyz="-0.675 0.8375 0.02" rpy="0 0 0"/>
+    <geometry>
+      <mesh filename="file://$(find car)/meshes/direction_front_right_1.stl" scale="0.001 0.001 0.001"/>
+    </geometry>
+    <material name="silver"/>
+  </visual>
+  <collision>
+    <origin xyz="-0.675 0.8375 0.02" rpy="0 0 0"/>
+    <geometry>
+      <mesh filename="file://$(find car)/meshes/direction_front_right_1.stl" scale="0.001 0.001 0.001"/>
+    </geometry>
+  </collision>
+</link>
+<link name="rim_front_right_1">
+  <inertial>
+    <origin xyz="-6.193392562137134e-07 -0.04445832186276233 -3.799540938658197e-06" rpy="0 0 0"/>
+    <mass value="35.2612545549612"/>
+    <inertia ixx="0.833786" iyy="1.48872" izz="0.833785" ixy="-1e-06" iyz="-3e-06" ixz="-3e-06"/>
+  </inertial>
+  <visual>
+    <origin xyz="-0.675 1.0 -0.0" rpy="0 0 0"/>
+    <geometry>
+      <mesh filename="file://$(find car)/meshes/rim_front_right_1.stl" scale="0.001 0.001 0.001"/>
+    </geometry>
+    <material name="silver"/>
+  </visual>
+  <collision>
+    <origin xyz="-0.675 1.0 -0.0" rpy="0 0 0"/>
+    <geometry>
+      <mesh filename="file://$(find car)/meshes/rim_front_right_1.stl" scale="0.001 0.001 0.001"/>
+    </geometry>
+  </collision>
+</link>
+<link name="tire_back_left_1">
+  <inertial>
+    <origin xyz="-4.773959005888173e-15 1.865424268387983e-07 1.7763568394002505e-15" rpy="0 0 0"/>
+    <mass value="72.8155229435052"/>
+    <inertia ixx="4.088543" iyy="7.430415" izz="4.088543" ixy="0.0" iyz="-0.0" ixz="0.0"/>
+  </inertial>
+  <visual>
+    <origin xyz="-0.675 1.047622 -0.0" rpy="0 0 0"/>
+    <geometry>
+      <mesh filename="file://$(find car)/meshes/tire_back_left_1.stl" scale="0.001 0.001 0.001"/>
+    </geometry>
+    <material name="silver"/>
+  </visual>
+  <collision>
+    <origin xyz="-0.675 1.047622 -0.0" rpy="0 0 0"/>
+    <geometry>
+      <mesh filename="file://$(find car)/meshes/tire_back_left_1.stl" scale="0.001 0.001 0.001"/>
+    </geometry>
+  </collision>
+</link>
+<link name="suspension_back_right_1">
+  <inertial>
+    <origin xyz="0.02499999999999991 -0.4032961129921663 0.0" rpy="0 0 0"/>
+    <mass value="33.21861256094089"/>
+    <inertia ixx="1.897101" iyy="0.053443" izz="1.887366" ixy="0.0" iyz="0.0" ixz="0.0"/>
+  </inertial>
+  <visual>
+    <origin xyz="0.7 0.125 -0.0" rpy="0 0 0"/>
+    <geometry>
+      <mesh filename="file://$(find car)/meshes/suspension_back_right_1.stl" scale="0.001 0.001 0.001"/>
+    </geometry>
+    <material name="silver"/>
+  </visual>
+  <collision>
+    <origin xyz="0.7 0.125 -0.0" rpy="0 0 0"/>
+    <geometry>
+      <mesh filename="file://$(find car)/meshes/suspension_back_right_1.stl" scale="0.001 0.001 0.001"/>
+    </geometry>
+  </collision>
+</link>
+<link name="direction_back_right_1">
+  <inertial>
+    <origin xyz="0.002014722651420331 -0.07474229529205345 0.02" rpy="0 0 0"/>
+    <mass value="11.386858894419664"/>
+    <inertia ixx="0.054235" iyy="0.024154" izz="0.06804" ixy="0.00144" iyz="0.0" ixz="-0.0"/>
+  </inertial>
+  <visual>
+    <origin xyz="0.675 0.8375 0.02" rpy="0 0 0"/>
+    <geometry>
+      <mesh filename="file://$(find car)/meshes/direction_back_right_1.stl" scale="0.001 0.001 0.001"/>
+    </geometry>
+    <material name="silver"/>
+  </visual>
+  <collision>
+    <origin xyz="0.675 0.8375 0.02" rpy="0 0 0"/>
+    <geometry>
+      <mesh filename="file://$(find car)/meshes/direction_back_right_1.stl" scale="0.001 0.001 0.001"/>
+    </geometry>
+  </collision>
+</link>
+<link name="rim_back_left_1">
+  <inertial>
+    <origin xyz="-6.193390665876208e-07 -0.04445832186276344 -3.799540942353019e-06" rpy="0 0 0"/>
+    <mass value="35.261254554957446"/>
+    <inertia ixx="0.833786" iyy="1.48872" izz="0.833785" ixy="-1e-06" iyz="-3e-06" ixz="-3e-06"/>
+  </inertial>
+  <visual>
+    <origin xyz="0.67 1.0 -0.0" rpy="0 0 0"/>
+    <geometry>
+      <mesh filename="file://$(find car)/meshes/rim_back_left_1.stl" scale="0.001 0.001 0.001"/>
+    </geometry>
+    <material name="silver"/>
+  </visual>
+  <collision>
+    <origin xyz="0.67 1.0 -0.0" rpy="0 0 0"/>
+    <geometry>
+      <mesh filename="file://$(find car)/meshes/rim_back_left_1.stl" scale="0.001 0.001 0.001"/>
+    </geometry>
+  </collision>
+</link>
+<link name="tire_back_right_1">
+  <inertial>
+    <origin xyz="-9.325873406851315e-15 1.8654242439630764e-07 1.7053025658242404e-15" rpy="0 0 0"/>
+    <mass value="72.81552294350364"/>
+    <inertia ixx="4.088543" iyy="7.430415" izz="4.088543" ixy="0.0" iyz="-0.0" ixz="0.0"/>
+  </inertial>
+  <visual>
+    <origin xyz="0.67 1.047622 -0.0" rpy="0 0 0"/>
+    <geometry>
+      <mesh filename="file://$(find car)/meshes/tire_back_right_1.stl" scale="0.001 0.001 0.001"/>
+    </geometry>
+    <material name="silver"/>
+  </visual>
+  <collision>
+    <origin xyz="0.67 1.047622 -0.0" rpy="0 0 0"/>
+    <geometry>
+      <mesh filename="file://$(find car)/meshes/tire_back_right_1.stl" scale="0.001 0.001 0.001"/>
+    </geometry>
+  </collision>
+</link>
+<link name="suspension_back_left_1">
+  <inertial>
+    <origin xyz="-0.025000000000000022 0.4032961129921663 0.0" rpy="0 0 0"/>
     <mass value="33.2186125609409"/>
     <inertia ixx="1.897101" iyy="0.053443" izz="1.887366" ixy="0.0" iyz="0.0" ixz="-0.0"/>
   </inertial>
   <visual>
-    <origin xyz="-1.925 -0.875 0.45" rpy="0 0 0"/>
-    <geometry>
-      <mesh filename="file://$(find car)/meshes/suspension_front_left__1.stl" scale="0.001 0.001 0.001"/>
-    </geometry>
-    <material name="silver"/>
-  </visual>
-  <collision>
-    <origin xyz="-1.925 -0.875 0.45" rpy="0 0 0"/>
-    <geometry>
-      <mesh filename="file://$(find car)/meshes/suspension_front_left__1.stl" scale="0.001 0.001 0.001"/>
-    </geometry>
-  </collision>
-</link>
-<link name="suspension_back_right_1">
-  <inertial>
-    <origin xyz="0.0 -0.4032961129921663 0.0" rpy="0 0 0"/>
-    <mass value="33.21861256094089"/>
-    <inertia ixx="1.897101" iyy="0.053443" izz="1.887366" ixy="0.0" iyz="0.0" ixz="0.0"/>
-  </inertial>
-  <visual>
-    <origin xyz="-0.575 -0.625 0.45" rpy="0 0 0"/>
-    <geometry>
-      <mesh filename="file://$(find car)/meshes/suspension_back_right_1.stl" scale="0.001 0.001 0.001"/>
-    </geometry>
-    <material name="silver"/>
-  </visual>
-  <collision>
-    <origin xyz="-0.575 -0.625 0.45" rpy="0 0 0"/>
-    <geometry>
-      <mesh filename="file://$(find car)/meshes/suspension_back_right_1.stl" scale="0.001 0.001 0.001"/>
-    </geometry>
-  </collision>
-</link>
-<link name="suspension_back_left_1">
-  <inertial>
-    <origin xyz="1.1102230246251565e-16 0.40329611299216617 0.0" rpy="0 0 0"/>
-    <mass value="33.2186125609409"/>
-    <inertia ixx="1.897101" iyy="0.053443" izz="1.887366" ixy="0.0" iyz="0.0" ixz="-0.0"/>
-  </inertial>
-  <visual>
-    <origin xyz="-0.575 -0.875 0.45" rpy="0 0 0"/>
+    <origin xyz="0.65 -0.125 -0.0" rpy="0 0 0"/>
     <geometry>
       <mesh filename="file://$(find car)/meshes/suspension_back_left_1.stl" scale="0.001 0.001 0.001"/>
@@ -100,5 +300,5 @@
   </visual>
   <collision>
-    <origin xyz="-0.575 -0.875 0.45" rpy="0 0 0"/>
+    <origin xyz="0.65 -0.125 -0.0" rpy="0 0 0"/>
     <geometry>
       <mesh filename="file://$(find car)/meshes/suspension_back_left_1.stl" scale="0.001 0.001 0.001"/>
@@ -106,32 +306,32 @@
   </collision>
 </link>
-<link name="rim_back_left_1">
-  <inertial>
-    <origin xyz="-6.193390665876208e-07 0.04445832186276344 3.799540942373003e-06" rpy="0 0 0"/>
-    <mass value="35.261254554957446"/>
+<link name="direction_back_left_1">
+  <inertial>
+    <origin xyz="0.002014722651420331 0.07474229529205356 -0.02" rpy="0 0 0"/>
+    <mass value="11.386858894419678"/>
+    <inertia ixx="0.054235" iyy="0.024154" izz="0.06804" ixy="-0.00144" iyz="0.0" ixz="0.0"/>
+  </inertial>
+  <visual>
+    <origin xyz="0.675 -0.8375 -0.02" rpy="0 0 0"/>
+    <geometry>
+      <mesh filename="file://$(find car)/meshes/direction_back_left_1.stl" scale="0.001 0.001 0.001"/>
+    </geometry>
+    <material name="silver"/>
+  </visual>
+  <collision>
+    <origin xyz="0.675 -0.8375 -0.02" rpy="0 0 0"/>
+    <geometry>
+      <mesh filename="file://$(find car)/meshes/direction_back_left_1.stl" scale="0.001 0.001 0.001"/>
+    </geometry>
+  </collision>
+</link>
+<link name="rim_back_right_1">
+  <inertial>
+    <origin xyz="-6.193391306474894e-07 0.04445832186276366 3.7995409559243855e-06" rpy="0 0 0"/>
+    <mass value="35.26125455495827"/>
     <inertia ixx="0.833786" iyy="1.48872" izz="0.833785" ixy="1e-06" iyz="-3e-06" ixz="3e-06"/>
   </inertial>
   <visual>
-    <origin xyz="-0.58 -1.75 0.45" rpy="0 0 0"/>
-    <geometry>
-      <mesh filename="file://$(find car)/meshes/rim_back_left_1.stl" scale="0.001 0.001 0.001"/>
-    </geometry>
-    <material name="silver"/>
-  </visual>
-  <collision>
-    <origin xyz="-0.58 -1.75 0.45" rpy="0 0 0"/>
-    <geometry>
-      <mesh filename="file://$(find car)/meshes/rim_back_left_1.stl" scale="0.001 0.001 0.001"/>
-    </geometry>
-  </collision>
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