Commit message: model full conected

File: workspace_full_conected/src/car_python/urdf/car.xacro (robot description, xacro)
@@ -364,4 +364,44 @@
   </collision>
 </link>
+<link name="Component24_1">
+  <inertial>
+    <origin xyz="-6.661338147750939e-16 1.1102230246251565e-16 0.050000000000000266" rpy="0 0 0"/>
+    <mass value="24.661502330679863"/>
+    <inertia ixx="0.082205" iyy="0.082205" izz="0.123308" ixy="0.0" iyz="-0.0" ixz="0.0"/>
+  </inertial>
+  <visual>
+    <origin xyz="-1.85 -0.75 -0.65" rpy="0 0 0"/>
+    <geometry>
+      <mesh filename="file://$(find car_description)/meshes/Component24_1.stl" scale="0.001 0.001 0.001"/>
+    </geometry>
+    <material name="silver"/>
+  </visual>
+  <collision>
+    <origin xyz="-1.85 -0.75 -0.65" rpy="0 0 0"/>
+    <geometry>
+      <mesh filename="file://$(find car_description)/meshes/Component24_1.stl" scale="0.001 0.001 0.001"/>
+    </geometry>
+  </collision>
+</link>
+<link name="Component25_1">
+  <inertial>
+    <origin xyz="0.004642800215263865 0.0 0.0018567355153457643" rpy="0 0 0"/>
+    <mass value="2.3549999999999622"/>
+    <inertia ixx="0.019357" iyy="0.001982" izz="0.01795" ixy="-0.0" iyz="-0.0" ixz="0.00067"/>
+  </inertial>
+  <visual>
+    <origin xyz="-2.175082 -0.75 -0.43922" rpy="0 0 0"/>
+    <geometry>
+      <mesh filename="file://$(find car_description)/meshes/Component25_1.stl" scale="0.001 0.001 0.001"/>
+    </geometry>
+    <material name="silver"/>
+  </visual>
+  <collision>
+    <origin xyz="-2.175082 -0.75 -0.43922" rpy="0 0 0"/>
+    <geometry>
+      <mesh filename="file://$(find car_description)/meshes/Component25_1.stl" scale="0.001 0.001 0.001"/>
+    </geometry>
+  </collision>
+</link>
 <joint name="Revolute 1" type="revolute">
   <origin xyz="1.925 0.625 -0.45" rpy="0 0 0"/>
@@ -469,3 +509,13 @@
   <child link="chasis_1"/>
 </joint>
+<joint name="Rigid 22" type="fixed">
+  <origin xyz="0.6 0.0 1.05" rpy="0 0 0"/>
+  <parent link="chasis_1"/>
+  <child link="Component24_1"/>
+</joint>
+<joint name="Rigid 23" type="fixed">
+  <origin xyz="0.925082 0.0 0.83922" rpy="0 0 0"/>
+  <parent link="chasis_1"/>
+  <child link="Component25_1"/>
+</joint>
 </robot>

Commit message: working in create walls for navigation

File: workspace_full_conected/src/car_python/urdf/car.xacro (robot description, xacro)
@@ -8,5 +8,5 @@
 <link name="base_link">
   <inertial>
-    <origin xyz="1.2499999999999998 0.75 -0.45" rpy="0 0 0"/>
+    <origin xyz="0 0 0" rpy="0 0 0"/>
     <mass value="195.94086385796686"/>
     <inertia ixx="0.825102" iyy="42.139945" izz="42.62574" ixy="-0.0" iyz="0.0" ixz="0.0"/>

File: workspace_full_conected/src/car_python/urdf/lidar.plugin.xacro (robot description, xacro)
@@ -17,6 +17,6 @@
             <!-- Define un barrido vertical; ajusta samples y ángulos según el FOV deseado -->
             <samples>16</samples>
-            <min_angle>-0.2618</min_angle>  <!-- -15° -->
-            <max_angle>0.2618</max_angle>    <!-- 15° -->
+            <min_angle>-0.523599</min_angle>  <!-- -15° -->
+            <max_angle>0.523599</max_angle>    <!-- 15° -->
           </vertical>
         </scan>
